Commit message: copyrights and clean

File: youbot_description/gazebo/gazebo.urdf.xacro (robot description, xacro)
@@ -1,4 +1,4 @@
 <?xml version="1.0"?>
-<!-- Refactored by Arn-O -->
+<!-- Copyright 2013 Arn-O. See the LICENSE file at the top-level directory of this distribution and at https://github.com/Arn-O/youbot_ros_tools/blob/master/LICENSE. -->
 <robot name="youbot" xmlns:xacro="http://ros.org/wiki/xacro">
   <gazebo>

File: youbot_description/urdf/spec.urdf.xacro (robot description, xacro)
@@ -1,4 +1,4 @@
 <?xml version="1.0"?>
-<!-- Refactored by Arn-O -->
+<!-- Copyright 2013 Arn-O. See the LICENSE file at the top-level directory of this distribution and at https://github.com/Arn-O/youbot_ros_tools/blob/master/LICENSE. -->
 <robot name="youbot" xmlns:xacro="http://www.ros.org/wiki/xacro">
   <!-- base -->

File: youbot_description/urdf/youbot.urdf.xacro (robot description, xacro)
@@ -1,4 +1,4 @@
 <?xml version="1.0"?>
-<!-- Refactored by Arn-O -->
+<!-- Copyright 2013 Arn-O. See the LICENSE file at the top-level directory of this distribution and at https://github.com/Arn-O/youbot_ros_tools/blob/master/LICENSE. -->
 <robot xmlns:xacro="http://www.ros.org/wiki/xacro" name="youbot">
   <xacro:property name="M_PI" value="3.1415926535897931"/>
@@ -273,5 +273,6 @@
       <child link="finger_left_link"/>
       <axis xyz="${finger_left_axis}"/>
-      <limit lower="${finger_left_limit_min}" upper="${finger_left_limit_max}" effort="${finger_joint_effort}" velocity="${finger_joint_velocity}"/>
+      <limit lower="${finger_left_limit_min}" upper="${finger_left_limit_max}"
+             effort="${finger_joint_effort}" velocity="${finger_joint_velocity}"/>
     </joint>
     <transmission name="tran6">
