Commit message: arm chain

File: youbot_description/urdf/spec.urdf.xacro (robot description, xacro)
@@ -22,15 +22,17 @@
   <xacro:property name="wheel_br_pose_y" value="-0.158" />
   <xacro:property name="wheel_br_pose_z" value="-0.034" />
-  <!-- wheels -->
+  <!-- plate -->
   <xacro:property name="plate_mass" value="2.397" />
   <xacro:property name="plate_pose_x" value="-0.159" />
   <xacro:property name="plate_pose_y" value="0.000" />
   <xacro:property name="plate_pose_z" value="0.046" />
-  <!-- arm -->
+  <!-- arm base -->
   <xacro:property name="arm_base_mass" value="0.961" />
   <xacro:property name="arm_base_pose_x" value="0.143" />
   <xacro:property name="arm_base_pose_y" value="0.000" />
   <xacro:property name="arm_base_pose_z" value="0.046" />
-  <xacro:property name="arm_1_link_mass" value="1.390" />
+  <xacro:property name="arm_joint_effort" value="1000" />
+  <xacro:property name="arm_joint_velocity" value="${M_PI * (90 / 180)}" />
+  <!-- arm_1 -->
   <xacro:property name="arm_1_link_pose_x" value="0.024" />
   <xacro:property name="arm_1_link_pose_y" value="0.000" />
@@ -39,10 +41,51 @@
   <xacro:property name="arm_1_link_orient_p" value="${M_PI * (0 / 180)}" />
   <xacro:property name="arm_1_link_orient_r" value="${M_PI * (180 / 180)}" />
-  <xacro:property name="arm_2_link_mass" value="1.318" />
+  <xacro:property name="arm_1_axis" value="0 0 1" />
+  <xacro:property name="arm_1_limit_min" value="${M_PI * (-169 / 180) }" />
+  <xacro:property name="arm_1_limit_max" value="${M_PI * (169 / 180) }" />
+  <xacro:property name="arm_1_link_mass" value="1.390" />
+  <!-- arm_2 -->
   <xacro:property name="arm_2_link_pose_x" value="0.033" />
   <xacro:property name="arm_2_link_pose_y" value="0.000" />
   <xacro:property name="arm_2_link_pose_z" value="0.000" />
-  <xacro:property name="arm_2_link_orient_y" value="${M_PI * (-90 / 180)}" />
-  <xacro:property name="arm_2_link_orient_p" value="${M_PI * (0 / 180)}" />
+  <xacro:property name="arm_2_link_orient_y" value="${M_PI * (0 / 180)}" />
+  <xacro:property name="arm_2_link_orient_p" value="${M_PI * (90 / 180)}" />
   <xacro:property name="arm_2_link_orient_r" value="${M_PI * (90 / 180)}" />
+  <xacro:property name="arm_2_axis" value="0 0 1" />
+  <xacro:property name="arm_2_limit_min" value="${M_PI * (-65 / 180) }" />
+  <xacro:property name="arm_2_limit_max" value="${M_PI * (90 / 180) }" />
+  <xacro:property name="arm_2_link_mass" value="1.318" />
+  <!-- arm_3 -->
+  <xacro:property name="arm_3_link_pose_x" value="0.155" />
+  <xacro:property name="arm_3_link_pose_y" value="0.000" />
+  <xacro:property name="arm_3_link_pose_z" value="0.000" />
+  <xacro:property name="arm_3_link_orient_y" value="${M_PI * (-90 / 180)}" />
+  <xacro:property name="arm_3_link_orient_p" value="${M_PI * (0 / 180)}" />
+  <xacro:property name="arm_3_link_orient_r" value="${M_PI * (0 / 180)}" />
+  <xacro:property name="arm_3_axis" value="0 0 1" />
+  <xacro:property name="arm_3_limit_min" value="${M_PI * (-151 / 180) }" />
+  <xacro:property name="arm_3_limit_max" value="${M_PI * (146 / 180) }" />
+  <xacro:property name="arm_3_link_mass" value="0.821" />
+  <!-- arm_4 -->
+  <xacro:property name="arm_4_link_pose_x" value="0.000" />
+  <xacro:property name="arm_4_link_pose_y" value="0.135" />
+  <xacro:property name="arm_4_link_pose_z" value="0.000" />
+  <xacro:property name="arm_4_link_orient_y" value="${M_PI * (0 / 180)}" />
+  <xacro:property name="arm_4_link_orient_p" value="${M_PI * (0 / 180)}" />
+  <xacro:property name="arm_4_link_orient_r" value="${M_PI * (0 / 180)}" />
+  <xacro:property name="arm_4_axis" value="0 0 1" />
+  <xacro:property name="arm_4_limit_min" value="${M_PI * (-102.5 / 180) }" />
+  <xacro:property name="arm_4_limit_max" value="${M_PI * (102.5 / 180) }" />
+  <xacro:property name="arm_4_link_mass" value="0.769" />
+  <!-- arm_5 -->
+  <xacro:property name="arm_5_link_pose_x" value="0.000" />
+  <xacro:property name="arm_5_link_pose_y" value="0.114" />
+  <xacro:property name="arm_5_link_pose_z" value="0.000" />
+  <xacro:property name="arm_5_link_orient_y" value="${M_PI * (0 / 180)}" />
+  <xacro:property name="arm_5_link_orient_p" value="${M_PI * (0 / 180)}" />
+  <xacro:property name="arm_5_link_orient_r" value="${M_PI * (-90 / 180)}" />
+  <xacro:property name="arm_5_axis" value="0 0 -1" />
+  <xacro:property name="arm_5_limit_min" value="${M_PI * (-165 / 180) }" />
+  <xacro:property name="arm_5_limit_max" value="${M_PI * (165 / 180) }" />
+  <xacro:property name="arm_5_link_mass" value="0.687" />
 </robot>

File: youbot_description/urdf/youbot.urdf.xacro (robot description, xacro)
@@ -5,6 +5,6 @@
   <xacro:include filename="$(find youbot_description)/urdf/spec.urdf.xacro" />
   <xacro:macro name="youbot_description" >
-    <!-- ### links ### -->
-    <!-- base -->
+    <!-- ### base ### -->
+    <!-- footprint link -->
     <link name="base_footprint">
       <inertial>
@@ -18,4 +18,5 @@
       </visual>
     </link>
+    <!-- base link -->
    <link name="base_link">
       <inertial>
@@ -29,4 +30,11 @@
       </visual>
     </link>
+  <!-- base joint -->
+    <joint name="base_joint" type="fixed">
+      <origin xyz="${base_pose_x} ${base_pose_y} ${base_pose_z}" rpy="0 0 0" />
+      <parent link="base_footprint"/>
+      <child link="base_link" />
+    </joint>
+    <!-- ### wheels ### -->
     <!-- wheels -->
     <!-- TODO: replace the following 4 code blocks by macros -->
@@ -99,4 +107,26 @@
       </collision>
     </link>
+  <!-- wheels joints -->
+    <joint name="wheel_fl_joint" type="fixed">
+      <origin xyz="${wheel_fl_pose_x} ${wheel_fl_pose_y} ${wheel_fl_pose_z}" rpy="0 0 0" />
+      <parent link="base_link"/>
+      <child link="wheel_link_fl" />
+    </joint>
+    <joint name="wheel_fr_joint" type="fixed">
+      <origin xyz="${wheel_fr_pose_x} ${wheel_fr_pose_y} ${wheel_fr_pose_z}" rpy="0 0 0" />
+      <parent link="base_link"/>
+      <child link="wheel_link_fr" />
+    </joint>
+    <joint name="wheel_bl_joint" type="fixed">
+      <origin xyz="${wheel_bl_pose_x} ${wheel_bl_pose_y} ${wheel_bl_pose_z}" rpy="0 0 0" />
+      <parent link="base_link"/>
+      <child link="wheel_link_bl" />
+    </joint>
+    <joint name="wheel_br_joint" type="fixed">
+      <origin xyz="${wheel_br_pose_x} ${wheel_br_pose_y} ${wheel_br_pose_z}" rpy="0 0 0" />
+      <parent link="base_link"/>
+      <child link="wheel_link_br" />
+    </joint>
+  <!-- #### plate #### -->
   <!-- plate links -->
   <link name="plate_link">
@@ -111,4 +141,11 @@
     </visual>
   </link>
+  <!-- plate joint -->
+    <joint name="plate_joint" type="fixed">
+      <origin xyz="${plate_pose_x} ${plate_pose_y} ${plate_pose_z}" rpy="0 0 0" />
+      <parent link="base_link"/>
+      <child link="plate_link" />
+    </joint>
+  <!-- ### arm_base ### -->
   <!-- arm_base link -->
     <link name="arm_base_link">
@@ -123,64 +160,4 @@
       </visual>
     </link>
-  <!-- arm_1 link -->
-    <link name="arm_1_link">
-      <inertial>
-        <mass value="${arm_1_link_mass}" />
-        <inertia ixx="0.010" ixy="0.000" ixz="0.000" iyy="0.010" iyz="0.000" izz="0.010" />
-      </inertial>
-      <visual>
-        <origin xyz="0 0 0" rpy="${arm_1_link_orient_r} ${arm_1_link_orient_p} ${arm_1_link_orient_y}" />
-        <geometry>
-          <mesh filename="package://youbot_description/meshes/arm_joint_1.dae"/>
-        </geometry>
-      </visual>
-    </link>
-  <!-- arm_2 link -->
-    <link name="arm_2_link">
-      <inertial>
-        <mass value="${arm_2_link_mass}" />
-        <inertia ixx="0.010" ixy="0.000" ixz="0.000" iyy="0.010" iyz="0.000" izz="0.010" />
-      </inertial>
-      <visual>
-        <origin xyz="0 0 0" rpy="${arm_2_link_orient_r} ${arm_2_link_orient_p} ${arm_2_link_orient_y}" />
-        <geometry>
-          <mesh filename="package://youbot_description/meshes/arm_joint_2.dae"/>
-        </geometry>
-      </visual>
-    </link>
-    <!-- ### joints ### -->
-  <!-- base joint -->
-    <joint name="base_joint" type="fixed">
-      <origin xyz="${base_pose_x} ${base_pose_y} ${base_pose_z}" rpy="0 0 0" />
-      <parent link="base_footprint"/>
-      <child link="base_link" />
-    </joint>
-  <!-- wheels joints -->
-    <joint name="wheel_fl_joint" type="fixed">
-      <origin xyz="${wheel_fl_pose_x} ${wheel_fl_pose_y} ${wheel_fl_pose_z}" rpy="0 0 0" />
-      <parent link="base_link"/>
-      <child link="wheel_link_fl" />
-    </joint>
-    <joint name="wheel_fr_joint" type="fixed">
-      <origin xyz="${wheel_fr_pose_x} ${wheel_fr_pose_y} ${wheel_fr_pose_z}" rpy="0 0 0" />
-      <parent link="base_link"/>
-      <child link="wheel_link_fr" />
-    </joint>
-    <joint name="wheel_bl_joint" type="fixed">
-      <origin xyz="${wheel_bl_pose_x} ${wheel_bl_pose_y} ${wheel_bl_pose_z}" rpy="0 0 0" />
-      <parent link="base_link"/>
-      <child link="wheel_link_bl" />
-    </joint>
-    <joint name="wheel_br_joint" type="fixed">
-      <origin xyz="${wheel_br_pose_x} ${wheel_br_pose_y} ${wheel_br_pose_z}" rpy="0 0 0" />
-      <parent link="base_link"/>
-      <child link="wheel_link_br" />
-    </joint>
-<!-- plate joint -->
-    <joint name="plate_joint" type="fixed">
-      <origin xyz="${arm_base_pose_x} ${arm_base_pose_y} ${arm_base_pose_z}" rpy="0 0 0" />
-      <parent link="base_link"/>
-      <child link="plate_link" />
-    </joint>
   <!-- arm_base joint -->
     <joint name="arm_base_joint" type="fixed">
@@ -189,19 +166,119 @@
       <child link="arm_base_link" />
     </joint>
+  <!-- TODO: replace the next 5 code blocks by macro -->
+  <!-- ### arm_1 ### -->
+  <!-- arm_1 link -->
+    <link name="arm_1_link">
+      <inertial>
+        <mass value="${arm_1_link_mass}" />
+        <inertia ixx="0.010" ixy="0.000" ixz="0.000" iyy="0.010" iyz="0.000" izz="0.010" />
+      </inertial>
+      <visual>
+        <geometry>
+          <mesh filename="package://youbot_description/meshes/arm_joint_1.dae"/>
+        </geometry>
+      </visual>
+    </link>
   <!-- arm_1 joint -->
     <joint name="arm_1_joint" type="revolute">
-      <origin xyz="${arm_1_link_pose_x} ${arm_1_link_pose_y} ${arm_1_link_pose_z}" />
+      <origin xyz="${arm_1_link_pose_x} ${arm_1_link_pose_y} ${arm_1_link_pose_z}"
+              rpy="${arm_1_link_orient_r} ${arm_1_link_orient_p} ${arm_1_link_orient_y}" />
       <parent link="arm_base_link"/>
       <child link="arm_1_link" />
-      <axis xyz="0 0 1" />
-      <limit lower="-2.0" upper="2.0" effort="1000" velocity="3" />
-    </joint>
+      <axis xyz="${arm_1_axis}" />
+      <limit lower="${arm_1_limit_min}" upper="${arm_1_limit_max}"
+             effort="${arm_joint_effort}" velocity="${arm_joint_velocity}" />
+    </joint>
+  <!-- ### arm_2 ### -->
+  <!-- arm_2 link -->
+    <link name="arm_2_link">
+      <inertial>
+        <mass value="${arm_2_link_mass}" />
+        <inertia ixx="0.010" ixy="0.000" ixz="0.000" iyy="0.010" iyz="0.000" izz="0.010" />
+      </inertial>
+      <visual>
+        <geometry>
+          <mesh filename="package://youbot_description/meshes/arm_joint_2.dae"/>
+        </geometry>
+      </visual>
+    </link>
   <!-- arm_2 joint -->
     <joint name="arm_2_joint" type="revolute">
-      <origin xyz="${arm_2_link_pose_x} ${arm_2_link_pose_y} ${arm_2_link_pose_z}" />
+      <origin xyz="${arm_2_link_pose_x} ${arm_2_link_pose_y} ${arm_2_link_pose_z}"
+              rpy="${arm_2_link_orient_r} ${arm_2_link_orient_p} ${arm_2_link_orient_y}" />
       <parent link="arm_1_link"/>
       <child link="arm_2_link" />
-      <axis xyz="0 1 0" />
-      <limit lower="-2.0" upper="2.0" effort="1000" velocity="3" />
+      <axis xyz="${arm_2_axis}" />
+      <limit lower="${arm_2_limit_min}" upper="${arm_2_limit_max}"
+             effort="${arm_joint_effort}" velocity="${arm_joint_velocity}" />
+    </joint>
+  <!-- ### arm_3 ### -->
+  <!-- arm_3 link -->
+    <link name="arm_3_link">
+      <inertial>
+        <mass value="${arm_3_link_mass}" />
+        <inertia ixx="0.010" ixy="0.000" ixz="0.000" iyy="0.010" iyz="0.000" izz="0.010" />
+      </inertial>
+      <visual>
+        <geometry>
+          <mesh filename="package://youbot_description/meshes/arm_joint_3.dae"/>
+        </geometry>
+      </visual>
+    </link>
+  <!-- arm_3 joint -->
+    <joint name="arm_3_joint" type="revolute">
+      <origin xyz="${arm_3_link_pose_x} ${arm_3_link_pose_y} ${arm_3_link_pose_z}"
+              rpy="${arm_3_link_orient_r} ${arm_3_link_orient_p} ${arm_3_link_orient_y}" />
+      <parent link="arm_2_link"/>
+      <child link="arm_3_link" />
+      <axis xyz="${arm_3_axis}" />
+      <limit lower="${arm_3_limit_min}" upper="${arm_3_limit_max}"
+             effort="${arm_joint_effort}" velocity="${arm_joint_velocity}" />
+    </joint>
+  <!-- ### arm_4 ### -->
+  <!-- arm_4 link -->
+    <link name="arm_4_link">
+      <inertial>
+        <mass value="${arm_4_link_mass}" />
+        <inertia ixx="0.010" ixy="0.000" ixz="0.000" iyy="0.010" iyz="0.000" izz="0.010" />
+      </inertial>
+      <visual>
+        <geometry>
+          <mesh filename="package://youbot_description/meshes/arm_joint_4.dae"/>
+        </geometry>
+      </visual>
+    </link>
+  <!-- arm_4 joint -->
+    <joint name="arm_4_joint" type="revolute">
+      <origin xyz="${arm_4_link_pose_x} ${arm_4_link_pose_y} ${arm_4_link_pose_z}"
+              rpy="${arm_4_link_orient_r} ${arm_4_link_orient_p} ${arm_4_link_orient_y}" />
+      <parent link="arm_3_link"/>
+      <child link="arm_4_link" />
+      <axis xyz="${arm_4_axis}" />
+      <limit lower="${arm_4_limit_min}" upper="${arm_4_limit_max}"
+             effort="${arm_joint_effort}" velocity="${arm_joint_velocity}" />
+    </joint>
+  <!-- ### arm_5 ### -->
+  <!-- arm_5 link -->
+    <link name="arm_5_link">
+      <inertial>
+        <mass value="${arm_5_link_mass}" />
+        <inertia ixx="0.010" ixy="0.000" ixz="0.000" iyy="0.010" iyz="0.000" izz="0.010" />
+      </inertial>
+      <visual>
+        <geometry>
+          <mesh filename="package://youbot_description/meshes/arm_joint_5.dae"/>
+        </geometry>
+      </visual>
+    </link>
+  <!-- arm_5 joint -->
+    <joint name="arm_5_joint" type="revolute">
+      <origin xyz="${arm_5_link_pose_x} ${arm_5_link_pose_y} ${arm_5_link_pose_z}"
+              rpy="${arm_5_link_orient_r} ${arm_5_link_orient_p} ${arm_5_link_orient_y}" />
+      <parent link="arm_4_link"/>
+      <child link="arm_5_link" />
+      <axis xyz="${arm_5_axis}" />
+      <limit lower="${arm_5_limit_min}" upper="${arm_5_limit_max}"
+             effort="${arm_joint_effort}" velocity="${arm_joint_velocity}" />
     </joint>
   </xacro:macro>

Commit message: setup first controller

File: youbot_description/urdf/spec.urdf.xacro (robot description, xacro)
@@ -49,4 +49,5 @@
   <xacro:property name="arm_2_link_pose_y" value="0.000" />
   <xacro:property name="arm_2_link_pose_z" value="0.000" />
+  <!-- slightly different from the doc due to different conventions -->
   <xacro:property name="arm_2_link_orient_y" value="${M_PI * (0 / 180)}" />
   <xacro:property name="arm_2_link_orient_p" value="${M_PI * (90 / 180)}" />

File: youbot_description/urdf/youbot.urdf.xacro (robot description, xacro)
@@ -3,5 +3,8 @@
 <robot name="youbot" xmlns:xacro="http://www.ros.org/wiki/xacro">
   <xacro:property name="M_PI" value="3.1415926535897931" />
+  <!-- Import the spec provided by youBot store -->
   <xacro:include filename="$(find youbot_description)/urdf/spec.urdf.xacro" />
+  <!-- Import all Gazebo-customization elements, including Gazebo colors -->
+  <xacro:include filename="$(find youbot_description)/urdf/youbot.gazebo" />
   <xacro:macro name="youbot_description" >
     <!-- ### base ### -->
@@ -190,4 +193,12 @@
              effort="${arm_joint_effort}" velocity="${arm_joint_velocity}" />
     </joint>
+  <transmission name="tran1">
+    <type>transmission_interface/SimpleTransmission</type>
+    <joint name="arm_1_joint"/>
+    <actuator name="motor1">
+      <hardwareInterface>EffortJointInterface</hardwareInterface>
+      <mechanicalReduction>1</mechanicalReduction>
+    </actuator>
+  </transmission>
   <!-- ### arm_2 ### -->
   <!-- arm_2 link -->

Commit message: gripper and finger

File: youbot_description/urdf/spec.urdf.xacro (robot description, xacro)
@@ -23,14 +23,16 @@
   <xacro:property name="wheel_br_pose_z" value="-0.034" />
   <!-- plate -->
-  <xacro:property name="plate_mass" value="2.397" />
   <xacro:property name="plate_pose_x" value="-0.159" />
   <xacro:property name="plate_pose_y" value="0.000" />
   <xacro:property name="plate_pose_z" value="0.046" />
+  <xacro:property name="plate_mass" value="2.397" />
   <!-- arm base -->
-  <xacro:property name="arm_base_mass" value="0.961" />
   <xacro:property name="arm_base_pose_x" value="0.143" />
   <xacro:property name="arm_base_pose_y" value="0.000" />
   <xacro:property name="arm_base_pose_z" value="0.046" />
-  <xacro:property name="arm_joint_effort" value="1000" />
+  <xacro:property name="arm_base_mass" value="0.961" />
+  <!-- TODO: insert max effort joint by joint -->
+  <!-- arms parameter -->
+  <xacro:property name="arm_joint_effort" value="10" />
   <xacro:property name="arm_joint_velocity" value="${M_PI * (90 / 180)}" />
   <!-- arm_1 -->
@@ -90,3 +92,32 @@
   <xacro:property name="arm_5_limit_max" value="${M_PI * (165 / 180) }" />
   <xacro:property name="arm_5_link_mass" value="0.687" />
+  <!-- gripper_base -->
+  <xacro:property name="gripper_base_link_pose_x" value="0.000" />
+  <xacro:property name="gripper_base_link_pose_y" value="0.000" />
+  <xacro:property name="gripper_base_link_pose_z" value="0.057" />
+  <xacro:property name="gripper_base_link_orient_y" value="${M_PI * (180 / 180)}" />
+  <xacro:property name="gripper_base_link_orient_p" value="${M_PI * (0 / 180)}" />
+  <xacro:property name="gripper_base_link_orient_r" value="${M_PI * (0 / 180)}" />
+  <xacro:property name="gripper_base_link_mass" value="0.199" />
+  <!-- fingers paramaters -->
+  <xacro:property name="finger_joint_effort" value="10" />
+  <xacro:property name="finger_joint_velocity" value="1" />
+  <!-- finger_left -->
+  <xacro:property name="finger_left_link_pose_x" value="0.000" />
+  <xacro:property name="finger_left_link_pose_y" value="0.008" />
+  <xacro:property name="finger_left_link_pose_z" value="0.000" />
+  <xacro:property name="finger_left_axis" value="0 1 0" />
+  <!-- TODO: the max value should be a parameter of the robot -->
+  <xacro:property name="finger_left_limit_min" value="0" />
+  <xacro:property name="finger_left_limit_max" value="0.013" />
+  <xacro:property name="finger_left_link_mass" value="0.010" />
+  <!-- finger_right -->
+  <xacro:property name="finger_right_link_pose_x" value="0.000" />
+  <xacro:property name="finger_right_link_pose_y" value="-0.008" />
+  <xacro:property name="finger_right_link_pose_z" value="0.000" />
+  <xacro:property name="finger_right_axis" value="0 -1 0" />
+  <!-- TODO: the max value should be a parameter of the robot -->
+  <xacro:property name="finger_right_limit_min" value="0" />
+  <xacro:property name="finger_right_limit_max" value="0.013" />
+  <xacro:property name="finger_right_link_mass" value="0.010" />
 </robot>

File: youbot_description/urdf/youbot.urdf.xacro (robot description, xacro)
@@ -293,8 +293,71 @@
              effort="${arm_joint_effort}" velocity="${arm_joint_velocity}" />
     </joint>
+  <!-- ### gripper_base ### -->
+  <!-- gripper_base link -->
+    <link name="gripper_base_link">
+      <inertial>
+        <mass value="${gripper_base_link_mass}" />
+        <inertia ixx="0.010" ixy="0.000" ixz="0.000" iyy="0.010" iyz="0.000" izz="0.010" />
+      </inertial>
+      <visual>
+        <geometry>
+          <mesh filename="package://youbot_description/meshes/gripper_base_frame.dae"/>
+        </geometry>
+      </visual>
+    </link>
+  <!-- gripper_base joint -->
+    <joint name="gripper_base_joint" type="fixed">
+      <origin xyz="${gripper_base_link_pose_x} ${gripper_base_link_pose_y} ${gripper_base_link_pose_z}"
+              rpy="${gripper_base_link_orient_r} ${gripper_base_link_orient_p}
+                                            ${gripper_base_link_orient_y}" />
+      <parent link="arm_5_link"/>
+      <child link="gripper_base_link" />
+    </joint>
+  <!-- ### finger_left ### -->
+  <!-- finger_left link -->
+    <link name="finger_left_link">
+      <inertial>
+        <mass value="${finger_left_link_mass}" />
+        <inertia ixx="0.010" ixy="0.000" ixz="0.000" iyy="0.010" iyz="0.000" izz="0.010" />
+      </inertial>
+      <visual>
+        <geometry>
+          <mesh filename="package://youbot_description/meshes/gripper_left_finger.dae"/>
+        </geometry>
+      </visual>
+    </link>
+  <!-- finger_left joint -->
+    <joint name="finger_left_joint" type="prismatic">
+      <origin xyz="${finger_left_link_pose_x} ${finger_left_link_pose_y} ${finger_left_link_pose_z}" />
+      <parent link="gripper_base_link"/>
+      <child link="finger_left_link" />
+      <axis xyz="${finger_left_axis}" />
+      <limit lower="${finger_left_limit_min}" upper="${finger_left_limit_max}"
+             effort="${finger_joint_effort}" velocity="${finger_joint_velocity}" />
+    </joint>
+  <!-- ### finger_right ### -->
+  <!-- finger_right link -->
+    <link name="finger_right_link">
+      <inertial>
+        <mass value="${finger_right_link_mass}" />
+        <inertia ixx="0.010" ixy="0.000" ixz="0.000" iyy="0.010" iyz="0.000" izz="0.010" />
+      </inertial>
+      <visual>
+        <geometry>
+          <mesh filename="package://youbot_description/meshes/gripper_right_finger.dae"/>
+        </geometry>
+      </visual>
+    </link>
+  <!-- finger_right joint -->
+    <joint name="finger_right_joint" type="prismatic">
+      <origin xyz="${finger_right_link_pose_x} ${finger_right_link_pose_y}
+                                                       ${finger_right_link_pose_z}" />
+      <parent link="gripper_base_link"/>
+      <child link="finger_right_link" />
+      <axis xyz="${finger_right_axis}" />
+      <limit lower="${finger_right_limit_min}" upper="${finger_right_limit_max}"
+             effort="${finger_joint_effort}" velocity="${finger_joint_velocity}" />
+    </joint>
   </xacro:macro>
   <xacro:youbot_description />
-    <!-- extensions -->
-    <!-- uncomment for adding the controllers -->
-    <!-- xacro:youbot_arm_transmission /-->
 </robot>
