Commit message: macro for wheels

File: youbot_description/urdf/spec.urdf.xacro (robot description, xacro)
@@ -10,16 +10,7 @@
   <xacro:property name="wheel_mass" value="1.400" />
   <xacro:property name="wheel_radius" value="0.050" />
-  <xacro:property name="wheel_fl_pose_x" value="0.228" />
-  <xacro:property name="wheel_fl_pose_y" value="0.158" />
-  <xacro:property name="wheel_fl_pose_z" value="-0.034" />
-  <xacro:property name="wheel_fr_pose_x" value="0.228" />
-  <xacro:property name="wheel_fr_pose_y" value="-0.158" />
-  <xacro:property name="wheel_fr_pose_z" value="-0.034" />
-  <xacro:property name="wheel_bl_pose_x" value="-0.228" />
-  <xacro:property name="wheel_bl_pose_y" value="0.158" />
-  <xacro:property name="wheel_bl_pose_z" value="-0.034" />
-  <xacro:property name="wheel_br_pose_x" value="-0.228" />
-  <xacro:property name="wheel_br_pose_y" value="-0.158" />
-  <xacro:property name="wheel_br_pose_z" value="-0.034" />
+  <xacro:property name="wheel_pose_x" value="0.228" />
+  <xacro:property name="wheel_pose_y" value="0.158" />
+  <xacro:property name="wheel_pose_z" value="-0.034" />
   <!-- plate -->
   <xacro:property name="plate_pose_x" value="-0.159" />

File: youbot_description/urdf/youbot.urdf.xacro (robot description, xacro)
@@ -7,6 +7,6 @@
   <!-- Import all Gazebo-customization elements, including Gazebo colors -->
   <xacro:include filename="$(find youbot_description)/urdf/youbot.gazebo" />
-  <xacro:macro name="youbot_description" >
-    <!-- ### base ### -->
+  <xacro:macro name="base" >
+    <!-- #### base #### -->
     <!-- footprint link -->
     <link name="base_footprint">
@@ -38,96 +38,4 @@
       <parent link="base_footprint"/>
       <child link="base_link" />
-    </joint>
-    <!-- ### wheels ### -->
-    <!-- wheels -->
-    <!-- TODO: replace the following 4 code blocks by macros -->
-    <!-- front left wheel -->
-    <link name="wheel_link_fl">
-      <inertial>
-        <mass value="${wheel_mass}" />
-        <inertia  ixx="0.010" ixy="0.000" ixz="0.000" iyy="0.010" iyz="0.000" izz="0.010" />
-      </inertial>
-      <visual>
-        <geometry>
-          <sphere radius="${wheel_radius}" />
-        </geometry>
-      </visual>
-      <collision>
-        <geometry>
-          <sphere radius="${wheel_radius}" />
-        </geometry>
-      </collision>
-    </link>
-    <!-- front right wheel -->
-    <link name="wheel_link_fr">
-      <inertial>
-        <mass value="${wheel_mass}" />
-        <inertia  ixx="0.010" ixy="0.000" ixz="0.000" iyy="0.010" iyz="0.000" izz="0.010" />
-      </inertial>
-      <visual>
-        <geometry>
-          <sphere radius="${wheel_radius}" />
-        </geometry>
-      </visual>
-      <collision>
-        <geometry>
-          <sphere radius="${wheel_radius}" />
-        </geometry>
-      </collision>
-    </link>
-    <!-- back left wheel -->
-    <link name="wheel_link_bl">
-      <inertial>
-        <mass value="${wheel_mass}" />
-        <inertia  ixx="0.010" ixy="0.000" ixz="0.000" iyy="0.010" iyz="0.000" izz="0.010" />
-      </inertial>
-      <visual>
-        <geometry>
-          <sphere radius="${wheel_radius}" />
-        </geometry>
-      </visual>
-      <collision>
-        <geometry>
-          <sphere radius="${wheel_radius}" />
-        </geometry>
-      </collision>
-    </link>
-    <!-- back right wheel -->
-    <link name="wheel_link_br">
-      <inertial>
-        <mass value="${wheel_mass}" />
-        <inertia  ixx="0.010" ixy="0.000" ixz="0.000" iyy="0.010" iyz="0.000" izz="0.010" />
-      </inertial>
-      <visual>
-        <geometry>
-          <sphere radius="${wheel_radius}" />
-        </geometry>
-      </visual>
-      <collision>
-        <geometry>
-          <sphere radius="${wheel_radius}" />
-        </geometry>
-      </collision>
-    </link>
-  <!-- wheels joints -->
-    <joint name="wheel_fl_joint" type="fixed">
-      <origin xyz="${wheel_fl_pose_x} ${wheel_fl_pose_y} ${wheel_fl_pose_z}" rpy="0 0 0" />
-      <parent link="base_link"/>
-      <child link="wheel_link_fl" />
-    </joint>
-    <joint name="wheel_fr_joint" type="fixed">
-      <origin xyz="${wheel_fr_pose_x} ${wheel_fr_pose_y} ${wheel_fr_pose_z}" rpy="0 0 0" />
-      <parent link="base_link"/>
-      <child link="wheel_link_fr" />
-    </joint>
-    <joint name="wheel_bl_joint" type="fixed">
-      <origin xyz="${wheel_bl_pose_x} ${wheel_bl_pose_y} ${wheel_bl_pose_z}" rpy="0 0 0" />
-      <parent link="base_link"/>
-      <child link="wheel_link_bl" />
-    </joint>
-    <joint name="wheel_br_joint" type="fixed">
-      <origin xyz="${wheel_br_pose_x} ${wheel_br_pose_y} ${wheel_br_pose_z}" rpy="0 0 0" />
-      <parent link="base_link"/>
-      <child link="wheel_link_br" />
     </joint>
   <!-- #### plate #### -->
@@ -150,6 +58,31 @@
       <child link="plate_link" />
     </joint>
-  <!-- ### arm_base ### -->
-  <!-- arm_base link -->
+  </xacro:macro>
+  <xacro:macro name="wheels" params="position x y">
+    <!-- ### wheels ### -->
+    <link name="wheel_${position}_link">
+      <inertial>
+        <mass value="${wheel_mass}" />
+        <inertia  ixx="0.010" ixy="0.000" ixz="0.000" iyy="0.010" iyz="0.000" izz="0.010" />
+      </inertial>
+      <visual>
+        <geometry>
+          <sphere radius="${wheel_radius}" />
+        </geometry>
+      </visual>
+      <collision>
+        <geometry>
+          <sphere radius="${wheel_radius}" />
+        </geometry>
+      </collision>
+    </link>
+    <joint name="wheel_${position}_joint" type="fixed">
+      <origin xyz="${wheel_pose_x * x} ${wheel_pose_y * y} ${wheel_pose_z}" />
+      <parent link="base_link"/>
+      <child link="wheel_${position}_link" />
+    </joint>
+  </xacro:macro>
+  <xacro:macro name="arm_base" >
+  <!-- #### arm_base #### -->
     <link name="arm_base_link">
       <inertial>
@@ -163,5 +96,4 @@
       </visual>
     </link>
-  <!-- arm_base joint -->
     <joint name="arm_base_joint" type="fixed">
       <origin xyz="${arm_base_pose_x} ${arm_base_pose_y} ${arm_base_pose_z}" rpy="0 0 0" />
@@ -169,4 +101,6 @@
       <child link="arm_base_link" />
     </joint>
+  </xacro:macro>
+  <xacro:macro name="arm" >
   <!-- TODO: replace the next 5 code blocks by macro -->
   <!-- ### arm_1 ### -->
@@ -224,4 +158,12 @@
              effort="${arm_joint_effort}" velocity="${arm_joint_velocity}" />
     </joint>
+  <transmission name="tran2">
+    <type>transmission_interface/SimpleTransmission</type>
+    <joint name="arm_2_joint"/>
+    <actuator name="motor2">
+      <hardwareInterface>EffortJointInterface</hardwareInterface>
+      <mechanicalReduction>1</mechanicalReduction>
+    </actuator>
+  </transmission>
   <!-- ### arm_3 ### -->
   <!-- arm_3 link -->
@@ -247,4 +189,12 @@
              effort="${arm_joint_effort}" velocity="${arm_joint_velocity}" />
     </joint>
+  <transmission name="tran3">
+    <type>transmission_interface/SimpleTransmission</type>
+    <joint name="arm_3_joint"/>
+    <actuator name="motor3">
+      <hardwareInterface>EffortJointInterface</hardwareInterface>
+      <mechanicalReduction>1</mechanicalReduction>
+    </actuator>
+  </transmission>
   <!-- ### arm_4 ### -->
   <!-- arm_4 link -->
@@ -270,4 +220,12 @@
              effort="${arm_joint_effort}" velocity="${arm_joint_velocity}" />
     </joint>
+  <transmission name="tran4">
+    <type>transmission_interface/SimpleTransmission</type>
+    <joint name="arm_4_joint"/>
+    <actuator name="motor4">
+      <hardwareInterface>EffortJointInterface</hardwareInterface>
+      <mechanicalReduction>1</mechanicalReduction>
+    </actuator>
+  </transmission>
   <!-- ### arm_5 ### -->
   <!-- arm_5 link -->
@@ -293,4 +251,14 @@
              effort="${arm_joint_effort}" velocity="${arm_joint_velocity}" />
     </joint>
+  <transmission name="tran5">
+    <type>transmission_interface/SimpleTransmission</type>
+    <joint name="arm_5_joint"/>
+    <actuator name="motor5">
+      <hardwareInterface>EffortJointInterface</hardwareInterface>
+      <mechanicalReduction>1</mechanicalReduction>
+    </actuator>
+  </transmission>
+  </xacro:macro>
+  <xacro:macro name="gripper" >
   <!-- ### gripper_base ### -->
   <!-- gripper_base link -->
@@ -360,4 +328,11 @@
     </joint>
   </xacro:macro>
-  <xacro:youbot_description />
+  <xacro:base />
+  <xacro:wheels position="fl" x="1" y="-1"/>
+  <xacro:wheels position="fr" x="1" y="1"/>
+  <xacro:wheels position="bl" x="-1" y="-1"/>
+  <xacro:wheels position="br" x="-1" y="1"/>
+  <xacro:arm_base />
+  <xacro:arm />
+  <xacro:gripper />
 </robot>

Commit message: properties for inertia

File: youbot_description/urdf/spec.urdf.xacro (robot description, xacro)
@@ -3,8 +3,8 @@
 <robot name="youbot" xmlns:xacro="http://www.ros.org/wiki/xacro">
   <!-- base -->
-  <xacro:property name="base_mass" value="19.803" />
   <xacro:property name="base_pose_x" value="0.000" />
   <xacro:property name="base_pose_y" value="0.000" />
   <xacro:property name="base_pose_z" value="0.084" />
+  <xacro:property name="base_mass" value="19.803" />
   <!-- wheels -->
   <xacro:property name="wheel_mass" value="1.400" />
@@ -23,7 +23,5 @@
   <xacro:property name="arm_base_pose_z" value="0.046" />
   <xacro:property name="arm_base_mass" value="0.961" />
-  <!-- TODO: insert max effort joint by joint -->
   <!-- arms parameter -->
-  <xacro:property name="arm_joint_effort" value="10" />
   <xacro:property name="arm_joint_velocity" value="${M_PI * (90 / 180)}" />
   <!-- arm_1 -->
@@ -38,4 +36,9 @@
   <xacro:property name="arm_1_limit_max" value="${M_PI * (169 / 180) }" />
   <xacro:property name="arm_1_link_mass" value="1.390" />
+  <xacro:property name="arm_1_joint_effort" value="9.5" />
+  <xacro:macro name="arm_1_inertia" >
+    <origin xyz="0.015 0.004 0.031" rpy="${M_PI * (180 / 180)} ${M_PI * (20 / 180)} 0"/>
+    <inertia ixx="0.0029525" iyy="0.0060091" izz="0.0058821" ixy="0.000" iyz="0.000" ixz="0.000" />
+  </xacro:macro>
   <!-- arm_2 -->
   <xacro:property name="arm_2_link_pose_x" value="0.033" />
@@ -50,4 +53,9 @@
   <xacro:property name="arm_2_limit_max" value="${M_PI * (90 / 180) }" />
   <xacro:property name="arm_2_link_mass" value="1.318" />
+  <xacro:property name="arm_2_joint_effort" value="9.5" />
+  <xacro:macro name="arm_2_inertia" >
+    <origin xyz="0.114 0.015 -0.019" rpy="0 ${M_PI * (90 / 180)} ${M_PI * (-90 / 180)}"/>
+    <inertia ixx="0.0031145" iyy="0.0005843" izz="0.0031631" ixy="0.000" iyz="0.000" ixz="0.000" />
+  </xacro:macro>
   <!-- arm_3 -->
   <xacro:property name="arm_3_link_pose_x" value="0.155" />
@@ -61,4 +69,9 @@
   <xacro:property name="arm_3_limit_max" value="${M_PI * (146 / 180) }" />
   <xacro:property name="arm_3_link_mass" value="0.821" />
+  <xacro:property name="arm_3_joint_effort" value="6.0" />
+  <xacro:macro name="arm_3_inertia" >
+    <origin xyz="0.000 0.104 0.020" rpy="0 0 ${M_PI * (90 / 180)}"/>
+    <inertia ixx="0.00172767" iyy="0.00041967" izz="0.0018468" ixy="0.000" iyz="0.000" ixz="0.000" />
+  </xacro:macro>
   <!-- arm_4 -->
   <xacro:property name="arm_4_link_pose_x" value="0.000" />
@@ -72,4 +85,9 @@
   <xacro:property name="arm_4_limit_max" value="${M_PI * (102.5 / 180) }" />
   <xacro:property name="arm_4_link_mass" value="0.769" />
+  <xacro:property name="arm_4_joint_effort" value="2.0" />
+  <xacro:macro name="arm_4_inertia" >
+    <origin xyz="0.000 0.054 -0.025" rpy="0 ${M_PI * (180 / 180)} ${M_PI * (40 / 180)}"/>
+    <inertia ixx="0.0006764" iyy="0.0010573" izz="0.0006610" ixy="0.000" iyz="0.000" ixz="0.000" />
+  </xacro:macro>
   <!-- arm_5 -->
   <xacro:property name="arm_5_link_pose_x" value="0.000" />
@@ -83,4 +101,9 @@
   <xacro:property name="arm_5_limit_max" value="${M_PI * (165 / 180) }" />
   <xacro:property name="arm_5_link_mass" value="0.687" />
+  <xacro:property name="arm_5_joint_effort" value="1.0" />
+  <xacro:macro name="arm_5_inertia" >
+    <origin xyz="0.000 0.001 -0.016" rpy="0 ${M_PI * (90 / 180)} 0"/>
+    <inertia ixx="0.0001934" iyy="0.0001602" izz="0.0000689" ixy="0.000" iyz="0.000" ixz="0.000" />
+  </xacro:macro>
   <!-- gripper_base -->
   <xacro:property name="gripper_base_link_pose_x" value="0.000" />
@@ -91,4 +114,8 @@
   <xacro:property name="gripper_base_link_orient_r" value="${M_PI * (0 / 180)}" />
   <xacro:property name="gripper_base_link_mass" value="0.199" />
+  <xacro:macro name="gripper_base_inertia" >
+    <origin xyz="0.000 0.000 0.029" rpy="0 ${M_PI * (180 / 180)} ${M_PI * (90 / 180)}"/>
+    <inertia ixx="0.0002324" iyy="0.0003629" izz="0.0002067" ixy="0.000" iyz="0.000" ixz="0.000" />
+  </xacro:macro>
   <!-- fingers paramaters -->
   <xacro:property name="finger_joint_effort" value="10" />

File: youbot_description/urdf/youbot.urdf.xacro (robot description, xacro)
@@ -7,4 +7,5 @@
   <!-- Import all Gazebo-customization elements, including Gazebo colors -->
   <xacro:include filename="$(find youbot_description)/urdf/youbot.gazebo" />
+  <!-- TODO: change inertia of the base links and the wheels -->
   <xacro:macro name="base" >
     <!-- #### base #### -->
@@ -13,5 +14,5 @@
       <inertial>
         <mass value="0.001" />
-        <inertia ixx="0.010" ixy="0.000" ixz="0.000" iyy="0.010" iyz="0.000" izz="0.010" />
+        <inertia ixx="0.000001" ixy="0.000" ixz="0.000" iyy="0.000001" iyz="0.000" izz="0.000001" />
       </inertial>
       <visual>
@@ -25,5 +26,5 @@
       <inertial>
         <mass value="${base_mass}" />
-        <inertia ixx="1.000" ixy="0.000" ixz="0.000" iyy="1.000" iyz="0.000" izz="1.000" />
+        <inertia ixx="0.01" ixy="0.000" ixz="0.000" iyy="0.01" iyz="0.000" izz="0.01" />
       </inertial>
       <visual>
@@ -35,5 +36,5 @@
   <!-- base joint -->
     <joint name="base_joint" type="fixed">
-      <origin xyz="${base_pose_x} ${base_pose_y} ${base_pose_z}" rpy="0 0 0" />
+      <origin xyz="${base_pose_x} ${base_pose_y} ${base_pose_z}" />
       <parent link="base_footprint"/>
       <child link="base_link" />
@@ -44,5 +45,5 @@
     <inertial>
      <mass value="${plate_mass}"/>
-     <inertia ixx="0.01" ixy="0" ixz="0" iyy="0.01" iyz="0" izz="0.01" />
+     <inertia ixx="0.002" ixy="0" ixz="0" iyy="0.002" iyz="0" izz="0.002" />
     </inertial>
     <visual>
@@ -54,5 +55,5 @@
   <!-- plate joint -->
     <joint name="plate_joint" type="fixed">
-      <origin xyz="${plate_pose_x} ${plate_pose_y} ${plate_pose_z}" rpy="0 0 0" />
+      <origin xyz="${plate_pose_x} ${plate_pose_y} ${plate_pose_z}" />
       <parent link="base_link"/>
       <child link="plate_link" />
@@ -64,5 +65,5 @@
       <inertial>
         <mass value="${wheel_mass}" />
-        <inertia  ixx="0.010" ixy="0.000" ixz="0.000" iyy="0.010" iyz="0.000" izz="0.010" />
+        <inertia  ixx="0.0014" ixy="0.000" ixz="0.000" iyy="0.0014" iyz="0.000" izz="0.0014" />
       </inertial>
       <visual>
@@ -109,5 +110,5 @@
       <inertial>
         <mass value="${arm_1_link_mass}" />
-        <inertia ixx="0.010" ixy="0.000" ixz="0.000" iyy="0.010" iyz="0.000" izz="0.010" />
+        <xacro:arm_1_inertia />
       </inertial>
       <visual>
@@ -125,5 +126,5 @@
       <axis xyz="${arm_1_axis}" />
       <limit lower="${arm_1_limit_min}" upper="${arm_1_limit_max}"
-             effort="${arm_joint_effort}" velocity="${arm_joint_velocity}" />
+             effort="${arm_1_joint_effort}" velocity="${arm_joint_velocity}" />
     </joint>
   <transmission name="tran1">
@@ -140,5 +141,5 @@
       <inertial>
         <mass value="${arm_2_link_mass}" />
-        <inertia ixx="0.010" ixy="0.000" ixz="0.000" iyy="0.010" iyz="0.000" izz="0.010" />
+        <xacro:arm_2_inertia />
       </inertial>
       <visual>
@@ -156,5 +157,5 @@
       <axis xyz="${arm_2_axis}" />
       <limit lower="${arm_2_limit_min}" upper="${arm_2_limit_max}"
-             effort="${arm_joint_effort}" velocity="${arm_joint_velocity}" />
+             effort="${arm_2_joint_effort}" velocity="${arm_joint_velocity}" />
     </joint>
   <transmission name="tran2">
@@ -171,5 +172,5 @@
       <inertial>
         <mass value="${arm_3_link_mass}" />
-        <inertia ixx="0.010" ixy="0.000" ixz="0.000" iyy="0.010" iyz="0.000" izz="0.010" />
+        <xacro:arm_3_inertia />
       </inertial>
       <visual>
@@ -187,5 +188,5 @@
       <axis xyz="${arm_3_axis}" />
       <limit lower="${arm_3_limit_min}" upper="${arm_3_limit_max}"
-             effort="${arm_joint_effort}" velocity="${arm_joint_velocity}" />
+             effort="${arm_3_joint_effort}" velocity="${arm_joint_velocity}" />
     </joint>
   <transmission name="tran3">
@@ -202,5 +203,5 @@
       <inertial>
         <mass value="${arm_4_link_mass}" />
-        <inertia ixx="0.010" ixy="0.000" ixz="0.000" iyy="0.010" iyz="0.000" izz="0.010" />
+        <xacro:arm_4_inertia />
       </inertial>
       <visual>
@@ -218,5 +219,5 @@
       <axis xyz="${arm_4_axis}" />
       <limit lower="${arm_4_limit_min}" upper="${arm_4_limit_max}"
-             effort="${arm_joint_effort}" velocity="${arm_joint_velocity}" />
+             effort="${arm_4_joint_effort}" velocity="${arm_joint_velocity}" />
     </joint>
   <transmission name="tran4">
@@ -233,5 +234,5 @@
       <inertial>
         <mass value="${arm_5_link_mass}" />
-        <inertia ixx="0.010" ixy="0.000" ixz="0.000" iyy="0.010" iyz="0.000" izz="0.010" />
+        <xacro:arm_5_inertia />
       </inertial>
       <visual>
@@ -249,5 +250,5 @@
       <axis xyz="${arm_5_axis}" />
       <limit lower="${arm_5_limit_min}" upper="${arm_5_limit_max}"
-             effort="${arm_joint_effort}" velocity="${arm_joint_velocity}" />
+             effort="${arm_5_joint_effort}" velocity="${arm_joint_velocity}" />
     </joint>
   <transmission name="tran5">
@@ -266,5 +267,5 @@
       <inertial>
         <mass value="${gripper_base_link_mass}" />
-        <inertia ixx="0.010" ixy="0.000" ixz="0.000" iyy="0.010" iyz="0.000" izz="0.010" />
+        <xacro:gripper_base_inertia />
       </inertial>
       <visual>
@@ -287,5 +288,5 @@
       <inertial>
         <mass value="${finger_left_link_mass}" />
-        <inertia ixx="0.010" ixy="0.000" ixz="0.000" iyy="0.010" iyz="0.000" izz="0.010" />
+        <inertia ixx="0.00001" ixy="0.000" ixz="0.000" iyy="0.00001" iyz="0.00001" izz="0.00001" />
       </inertial>
       <visual>
@@ -304,4 +305,12 @@
              effort="${finger_joint_effort}" velocity="${finger_joint_velocity}" />
     </joint>
+  <transmission name="tran6">
+    <type>transmission_interface/SimpleTransmission</type>
+    <joint name="finger_left_joint"/>
+    <actuator name="motor6">
+      <hardwareInterface>EffortJointInterface</hardwareInterface>
+      <mechanicalReduction>1</mechanicalReduction>
+    </actuator>
+  </transmission>
   <!-- ### finger_right ### -->
   <!-- finger_right link -->
@@ -309,5 +318,5 @@
       <inertial>
         <mass value="${finger_right_link_mass}" />
-        <inertia ixx="0.010" ixy="0.000" ixz="0.000" iyy="0.010" iyz="0.000" izz="0.010" />
+        <inertia ixx="0.00001" ixy="0.000" ixz="0.000" iyy="0.00001" iyz="0.00001" izz="0.00001" />
       </inertial>
       <visual>
@@ -327,4 +336,12 @@
              effort="${finger_joint_effort}" velocity="${finger_joint_velocity}" />
     </joint>
+  <transmission name="tran7">
+    <type>transmission_interface/SimpleTransmission</type>
+    <joint name="finger_right_joint"/>
+    <actuator name="motor7">
+      <hardwareInterface>EffortJointInterface</hardwareInterface>
+      <mechanicalReduction>1</mechanicalReduction>
+    </actuator>
+  </transmission>
   </xacro:macro>
   <xacro:base />
