Commit message: blocks for arm

File: youbot_description/urdf/youbot.urdf.xacro (robot description, xacro)
@@ -1,30 +1,30 @@
 <?xml version="1.0"?>
 <!-- Refactored by Arn-O -->
-<robot name="youbot" xmlns:xacro="http://www.ros.org/wiki/xacro">
-  <xacro:property name="M_PI" value="3.1415926535897931" />
+<robot xmlns:xacro="http://www.ros.org/wiki/xacro" name="youbot">
+  <xacro:property name="M_PI" value="3.1415926535897931"/>
   <!-- Import the spec provided by youBot store -->
-  <xacro:include filename="$(find youbot_description)/urdf/spec.urdf.xacro" />
+  <xacro:include filename="$(find youbot_description)/urdf/spec.urdf.xacro"/>
   <!-- Import all Gazebo-customization elements, including Gazebo colors -->
-  <xacro:include filename="$(find youbot_description)/urdf/youbot.gazebo" />
+  <xacro:include filename="$(find youbot_description)/urdf/youbot.gazebo"/>
   <!-- TODO: change inertia of the base links and the wheels -->
-  <xacro:macro name="base" >
+  <xacro:macro name="base">
     <!-- #### base #### -->
     <!-- footprint link -->
     <link name="base_footprint">
       <inertial>
-        <mass value="0.001" />
-        <inertia ixx="0.000001" ixy="0.000" ixz="0.000" iyy="0.000001" iyz="0.000" izz="0.000001" />
-      </inertial>
-      <visual>
-        <geometry>
-          <box size="0.001 0.001 0.001" />
+        <mass value="0.001"/>
+        <inertia ixx="0.000001" ixy="0.000" ixz="0.000" iyy="0.000001" iyz="0.000" izz="0.000001"/>
+      </inertial>
+      <visual>
+        <geometry>
+          <box size="0.001 0.001 0.001"/>
         </geometry>
       </visual>
     </link>
     <!-- base link -->
-   <link name="base_link">
-      <inertial>
-        <mass value="${base_mass}" />
-        <inertia ixx="0.01" ixy="0.000" ixz="0.000" iyy="0.01" iyz="0.000" izz="0.01" />
+    <link name="base_link">
+      <inertial>
+        <mass value="${base_mass}"/>
+        <inertia ixx="0.01" ixy="0.000" ixz="0.000" iyy="0.01" iyz="0.000" izz="0.01"/>
       </inertial>
       <visual>
@@ -34,28 +34,28 @@
       </visual>
     </link>
-  <!-- base joint -->
+    <!-- base joint -->
     <joint name="base_joint" type="fixed">
-      <origin xyz="${base_pose_x} ${base_pose_y} ${base_pose_z}" />
+      <origin xyz="${base_pose_x} ${base_pose_y} ${base_pose_z}"/>
       <parent link="base_footprint"/>
-      <child link="base_link" />
-    </joint>
-  <!-- #### plate #### -->
-  <!-- plate links -->
-  <link name="plate_link">
-    <inertial>
-     <mass value="${plate_mass}"/>
-     <inertia ixx="0.002" ixy="0" ixz="0" iyy="0.002" iyz="0" izz="0.002" />
-    </inertial>
-    <visual>
-      <geometry>
-        <mesh filename="package://youbot_description/meshes/plate.dae" />
-      </geometry>
-    </visual>
-  </link>
-  <!-- plate joint -->
+      <child link="base_link"/>
+    </joint>
+    <!-- #### plate #### -->
+    <!-- plate links -->
+    <link name="plate_link">
+      <inertial>
+        <mass value="${plate_mass}"/>
+        <inertia ixx="0.002" ixy="0" ixz="0" iyy="0.002" iyz="0" izz="0.002"/>
+      </inertial>
+      <visual>
+        <geometry>
+          <mesh filename="package://youbot_description/meshes/plate.dae"/>
+        </geometry>
+      </visual>
+    </link>
+    <!-- plate joint -->
     <joint name="plate_joint" type="fixed">
-      <origin xyz="${plate_pose_x} ${plate_pose_y} ${plate_pose_z}" />
+      <origin xyz="${plate_pose_x} ${plate_pose_y} ${plate_pose_z}"/>
       <parent link="base_link"/>
-      <child link="plate_link" />
+      <child link="plate_link"/>
     </joint>
   </xacro:macro>
@@ -64,30 +64,30 @@
     <link name="wheel_${position}_link">
       <inertial>
-        <mass value="${wheel_mass}" />
-        <inertia  ixx="0.0014" ixy="0.000" ixz="0.000" iyy="0.0014" iyz="0.000" izz="0.0014" />
-      </inertial>
-      <visual>
-        <geometry>
-          <sphere radius="${wheel_radius}" />
+        <mass value="${wheel_mass}"/>
+        <inertia ixx="0.0014" ixy="0.000" ixz="0.000" iyy="0.0014" iyz="0.000" izz="0.0014"/>
+      </inertial>
+      <visual>
+        <geometry>
+          <sphere radius="${wheel_radius}"/>
         </geometry>
       </visual>
       <collision>
         <geometry>
-          <sphere radius="${wheel_radius}" />
+          <sphere radius="${wheel_radius}"/>
         </geometry>
       </collision>
     </link>
     <joint name="wheel_${position}_joint" type="fixed">
-      <origin xyz="${wheel_pose_x * x} ${wheel_pose_y * y} ${wheel_pose_z}" />
+      <origin xyz="${wheel_pose_x * x} ${wheel_pose_y * y} ${wheel_pose_z}"/>
       <parent link="base_link"/>
-      <child link="wheel_${position}_link" />
-    </joint>
-  </xacro:macro>
-  <xacro:macro name="arm_base" >
-  <!-- #### arm_base #### -->
+      <child link="wheel_${position}_link"/>
+    </joint>
+  </xacro:macro>
+  <xacro:macro name="arm_base">
+    <!-- #### arm_base #### -->
     <link name="arm_base_link">
       <inertial>
-        <mass value="${arm_base_mass}" />
-        <inertia ixx="0.010" ixy="0.000" ixz="0.000" iyy="0.010" iyz="0.000" izz="0.010" />
+        <mass value="${arm_base_mass}"/>
+        <inertia ixx="0.010" ixy="0.000" ixz="0.000" iyy="0.010" iyz="0.000" izz="0.010"/>
       </inertial>
       <visual>
@@ -98,17 +98,16 @@
     </link>
     <joint name="arm_base_joint" type="fixed">
-      <origin xyz="${arm_base_pose_x} ${arm_base_pose_y} ${arm_base_pose_z}" rpy="0 0 0" />
+      <origin xyz="${arm_base_pose_x} ${arm_base_pose_y} ${arm_base_pose_z}" rpy="0 0 0"/>
       <parent link="base_link"/>
-      <child link="arm_base_link" />
-    </joint>
-  </xacro:macro>
-  <xacro:macro name="arm" >
-  <!-- TODO: replace the next 5 code blocks by macro -->
-  <!-- ### arm_1 ### -->
-  <!-- arm_1 link -->
+      <child link="arm_base_link"/>
+    </joint>
+  </xacro:macro>
+  <!-- #### arm #### -->
+  <xacro:macro name="arm">
+    <!-- ### arm_1 ### -->
+    <!-- arm_1 link -->
     <link name="arm_1_link">
       <inertial>
-        <mass value="${arm_1_link_mass}" />
-        <xacro:arm_1_inertia />
+        <xacro:arm_1_inertial/>
       </inertial>
       <visual>
@@ -118,28 +117,22 @@
       </visual>
     </link>
-  <!-- arm_1 joint -->
+    <!-- arm_1 joint -->
     <joint name="arm_1_joint" type="revolute">
-      <origin xyz="${arm_1_link_pose_x} ${arm_1_link_pose_y} ${arm_1_link_pose_z}"
-              rpy="${arm_1_link_orient_r} ${arm_1_link_orient_p} ${arm_1_link_orient_y}" />
-      <parent link="arm_base_link"/>
-      <child link="arm_1_link" />
-      <axis xyz="${arm_1_axis}" />
-      <limit lower="${arm_1_limit_min}" upper="${arm_1_limit_max}"
-             effort="${arm_1_joint_effort}" velocity="${arm_joint_velocity}" />
-    </joint>
-  <transmission name="tran1">
-    <type>transmission_interface/SimpleTransmission</type>
-    <joint name="arm_1_joint"/>
-    <actuator name="motor1">
-      <hardwareInterface>EffortJointInterface</hardwareInterface>
-      <mechanicalReduction>1</mechanicalReduction>
-    </actuator>
-  </transmission>
-  <!-- ### arm_2 ### -->
-  <!-- arm_2 link -->
+      <xacro:arm_1_joint/>
+      <child link="arm_1_link"/>
+    </joint>
+    <transmission name="tran1">
+      <type>transmission_interface/SimpleTransmission</type>
+      <joint name="arm_1_joint"/>
+      <actuator name="motor1">
+        <hardwareInterface>EffortJointInterface</hardwareInterface>
+        <mechanicalReduction>1</mechanicalReduction>
+      </actuator>
+    </transmission>
+    <!-- ### arm_2 ### -->
+    <!-- arm_2 link -->
     <link name="arm_2_link">
       <inertial>
-        <mass value="${arm_2_link_mass}" />
-        <xacro:arm_2_inertia />
+        <xacro:arm_2_inertial/>
       </inertial>
       <visual>
@@ -149,28 +142,22 @@
       </visual>
     </link>
-  <!-- arm_2 joint -->
+    <!-- arm_2 joint -->
     <joint name="arm_2_joint" type="revolute">
-      <origin xyz="${arm_2_link_pose_x} ${arm_2_link_pose_y} ${arm_2_link_pose_z}"
-              rpy="${arm_2_link_orient_r} ${arm_2_link_orient_p} ${arm_2_link_orient_y}" />
-      <parent link="arm_1_link"/>
-      <child link="arm_2_link" />
-      <axis xyz="${arm_2_axis}" />
-      <limit lower="${arm_2_limit_min}" upper="${arm_2_limit_max}"
-             effort="${arm_2_joint_effort}" velocity="${arm_joint_velocity}" />
-    </joint>
-  <transmission name="tran2">
-    <type>transmission_interface/SimpleTransmission</type>
-    <joint name="arm_2_joint"/>
-    <actuator name="motor2">
-      <hardwareInterface>EffortJointInterface</hardwareInterface>
-      <mechanicalReduction>1</mechanicalReduction>
-    </actuator>
-  </transmission>
-  <!-- ### arm_3 ### -->
-  <!-- arm_3 link -->
+      <xacro:arm_2_joint/>
+      <child link="arm_2_link"/>
+    </joint>
+    <transmission name="tran2">
+      <type>transmission_interface/SimpleTransmission</type>
+      <joint name="arm_2_joint"/>
+      <actuator name="motor2">
+        <hardwareInterface>EffortJointInterface</hardwareInterface>
+        <mechanicalReduction>1</mechanicalReduction>
+      </actuator>
+    </transmission>
+    <!-- ### arm_3 ### -->
+    <!-- arm_3 link -->
     <link name="arm_3_link">
       <inertial>
-        <mass value="${arm_3_link_mass}" />
-        <xacro:arm_3_inertia />
+        <xacro:arm_3_inertial/>
       </inertial>
       <visual>
@@ -180,28 +167,22 @@
       </visual>
     </link>
-  <!-- arm_3 joint -->
+    <!-- arm_3 joint -->
     <joint name="arm_3_joint" type="revolute">
-      <origin xyz="${arm_3_link_pose_x} ${arm_3_link_pose_y} ${arm_3_link_pose_z}"
-              rpy="${arm_3_link_orient_r} ${arm_3_link_orient_p} ${arm_3_link_orient_y}" />
-      <parent link="arm_2_link"/>
-      <child link="arm_3_link" />
-      <axis xyz="${arm_3_axis}" />
-      <limit lower="${arm_3_limit_min}" upper="${arm_3_limit_max}"
-             effort="${arm_3_joint_effort}" velocity="${arm_joint_velocity}" />
-    </joint>
-  <transmission name="tran3">
-    <type>transmission_interface/SimpleTransmission</type>
-    <joint name="arm_3_joint"/>
-    <actuator name="motor3">
-      <hardwareInterface>EffortJointInterface</hardwareInterface>
-      <mechanicalReduction>1</mechanicalReduction>
-    </actuator>
-  </transmission>
-  <!-- ### arm_4 ### -->
-  <!-- arm_4 link -->
+      <xacro:arm_3_joint/>
+      <child link="arm_3_link"/>
+    </joint>
+    <transmission name="tran3">
+      <type>transmission_interface/SimpleTransmission</type>
+      <joint name="arm_3_joint"/>
+      <actuator name="motor3">
+        <hardwareInterface>EffortJointInterface</hardwareInterface>
+        <mechanicalReduction>1</mechanicalReduction>
+      </actuator>
+    </transmission>
+    <!-- ### arm_4 ### -->
+    <!-- arm_4 link -->
     <link name="arm_4_link">
       <inertial>
-        <mass value="${arm_4_link_mass}" />
-        <xacro:arm_4_inertia />
+        <xacro:arm_4_inertial/>
       </inertial>
       <visual>
@@ -211,28 +192,22 @@
       </visual>
     </link>
-  <!-- arm_4 joint -->
+    <!-- arm_4 joint -->
     <joint name="arm_4_joint" type="revolute">
-      <origin xyz="${arm_4_link_pose_x} ${arm_4_link_pose_y} ${arm_4_link_pose_z}"
-              rpy="${arm_4_link_orient_r} ${arm_4_link_orient_p} ${arm_4_link_orient_y}" />
-      <parent link="arm_3_link"/>
-      <child link="arm_4_link" />
-      <axis xyz="${arm_4_axis}" />
-      <limit lower="${arm_4_limit_min}" upper="${arm_4_limit_max}"
-             effort="${arm_4_joint_effort}" velocity="${arm_joint_velocity}" />
-    </joint>
-  <transmission name="tran4">
-    <type>transmission_interface/SimpleTransmission</type>
-    <joint name="arm_4_joint"/>
-    <actuator name="motor4">
-      <hardwareInterface>EffortJointInterface</hardwareInterface>
-      <mechanicalReduction>1</mechanicalReduction>
-    </actuator>
-  </transmission>
-  <!-- ### arm_5 ### -->
-  <!-- arm_5 link -->
+      <xacro:arm_4_joint/>
+      <child link="arm_4_link"/>
+    </joint>
+    <transmission name="tran4">
+      <type>transmission_interface/SimpleTransmission</type>
+      <joint name="arm_4_joint"/>
+      <actuator name="motor4">
+        <hardwareInterface>EffortJointInterface</hardwareInterface>
+        <mechanicalReduction>1</mechanicalReduction>
+      </actuator>
+    </transmission>
+    <!-- ### arm_5 ### -->
+    <!-- arm_5 link -->
     <link name="arm_5_link">
       <inertial>
-        <mass value="${arm_5_link_mass}" />
-        <xacro:arm_5_inertia />
+        <xacro:arm_5_inertial/>
       </inertial>
       <visual>
@@ -242,30 +217,25 @@
       </visual>
     </link>
-  <!-- arm_5 joint -->
+    <!-- arm_5 joint -->
     <joint name="arm_5_joint" type="revolute">
-      <origin xyz="${arm_5_link_pose_x} ${arm_5_link_pose_y} ${arm_5_link_pose_z}"
-              rpy="${arm_5_link_orient_r} ${arm_5_link_orient_p} ${arm_5_link_orient_y}" />
-      <parent link="arm_4_link"/>
-      <child link="arm_5_link" />
-      <axis xyz="${arm_5_axis}" />
-      <limit lower="${arm_5_limit_min}" upper="${arm_5_limit_max}"
-             effort="${arm_5_joint_effort}" velocity="${arm_joint_velocity}" />
-    </joint>
-  <transmission name="tran5">
-    <type>transmission_interface/SimpleTransmission</type>
-    <joint name="arm_5_joint"/>
-    <actuator name="motor5">
-      <hardwareInterface>EffortJointInterface</hardwareInterface>
-      <mechanicalReduction>1</mechanicalReduction>
-    </actuator>
-  </transmission>
-  </xacro:macro>
-  <xacro:macro name="gripper" >
-  <!-- ### gripper_base ### -->
-  <!-- gripper_base link -->
+      <xacro:arm_5_joint/>
+      <child link="arm_5_link"/>
+    </joint>
+    <transmission name="tran5">
+      <type>transmission_interface/SimpleTransmission</type>
+      <joint name="arm_5_joint"/>
+      <actuator name="motor5">
+        <hardwareInterface>EffortJointInterface</hardwareInterface>
+        <mechanicalReduction>1</mechanicalReduction>
+      </actuator>
+    </transmission>
+  </xacro:macro>
+  <xacro:macro name="gripper">
+    <!-- ### gripper_base ### -->
+    <!-- gripper_base link -->
     <link name="gripper_base_link">
       <inertial>
-        <mass value="${gripper_base_link_mass}" />
-        <xacro:gripper_base_inertia />
+        <mass value="${gripper_base_link_mass}"/>
+        <xacro:gripper_base_inertia/>
       </inertial>
       <visual>
@@ -275,18 +245,17 @@
       </visual>
     </link>
-  <!-- gripper_base joint -->
+    <!-- gripper_base joint -->
     <joint name="gripper_base_joint" type="fixed">
       <origin xyz="${gripper_base_link_pose_x} ${gripper_base_link_pose_y} ${gripper_base_link_pose_z}"
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
Commit message: correct max effort

File: youbot_description/urdf/spec.urdf.xacro (robot description, xacro)
@@ -32,5 +32,5 @@
     <axis xyz="0 0 1" />
     <limit lower="${M_PI * (-169 / 180) }" upper="${M_PI * (169 / 180) }"
-           effort="9.5" velocity="${arm_joint_velocity}" />
+           effort="${9.5 * effort_correct}" velocity="${arm_joint_velocity}" />
   </xacro:macro>
   <xacro:macro name="arm_1_inertial" >
@@ -49,5 +49,5 @@
     <axis xyz="0 0 1" />
     <limit lower="${M_PI * (-65 / 180) }" upper="${M_PI * (90 / 180) }"
-           effort="9.5" velocity="${arm_joint_velocity}" />
+           effort="${9.5 * effort_correct}" velocity="${arm_joint_velocity}" />
   </xacro:macro>
   <xacro:macro name="arm_2_inertial" >
@@ -65,5 +65,5 @@
     <axis xyz="0 0 1" />
     <limit lower="${M_PI * (-151 / 180) }" upper="${M_PI * (146 / 180) }"
-           effort="6.0" velocity="${arm_joint_velocity}" />
+           effort="${6.0 * effort_correct}" velocity="${arm_joint_velocity}" />
   </xacro:macro>
   <xacro:macro name="arm_3_inertial" >
@@ -81,5 +81,5 @@
     <axis xyz="0 0 1" />
     <limit lower="${M_PI * (-102.5 / 180) }" upper="${M_PI * (102.5 / 180) }"
-           effort="10.0" velocity="${arm_joint_velocity}" />
+           effort="${2.0 * effort_correct}" velocity="${arm_joint_velocity}" />
   </xacro:macro>
   <xacro:macro name="arm_4_inertial" >
@@ -97,5 +97,5 @@
     <axis xyz="0 0 -1" />
     <limit lower="${M_PI * (-165 / 180) }" upper="${M_PI * (165 / 180) }"
-           effort="10.0" velocity="${arm_joint_velocity}" />
+           effort="${1.0 * effort_correct}" velocity="${arm_joint_velocity}" />
   </xacro:macro>
   <xacro:macro name="arm_5_inertial" >

File: youbot_description/urdf/youbot.urdf.xacro (robot description, xacro)
@@ -3,4 +3,6 @@
 <robot xmlns:xacro="http://www.ros.org/wiki/xacro" name="youbot">
   <xacro:property name="M_PI" value="3.1415926535897931"/>
+  <!-- used for having a more realistic behavior -->
+  <xacro:property name="effort_correct" value="10.0" />
   <!-- Import the spec provided by youBot store -->
   <xacro:include filename="$(find youbot_description)/urdf/spec.urdf.xacro"/>

Commit message: bug on inertia

File: youbot_description/urdf/spec.urdf.xacro (robot description, xacro)
@@ -36,8 +36,10 @@
   <xacro:macro name="arm_1_inertial" >
     <mass value="1.390" />
-    <origin xyz="0.015 0.004 0.031"
+    <inertia ixx="0.001" iyy="0.001" izz="0.001"
+             ixy="0.000" iyz="0.000" ixz="0.000" />
+    <!-- origin xyz="0.015 0.004 0.031"
             rpy="${M_PI * (180 / 180)} ${M_PI * (20 / 180)} 0"/>
     <inertia ixx="0.0029525" iyy="0.0060091" izz="0.0058821"
-             ixy="0.000" iyz="0.000" ixz="0.000" />
+             ixy="0.000" iyz="0.000" ixz="0.000" /-->
   </xacro:macro>
   <!-- arm_2 -->
@@ -53,8 +55,10 @@
   <xacro:macro name="arm_2_inertial" >
     <mass value="1.318" />
-    <origin xyz="0.114 0.015 -0.019"
+    <inertia ixx="0.001" iyy="0.001" izz="0.001"
+             ixy="0.000" iyz="0.000" ixz="0.000" />
+    <!-- origin xyz="0.114 0.015 -0.019"
             rpy="0 ${M_PI * (90 / 180)} ${M_PI * (-90 / 180)}"/>
     <inertia ixx="0.0031145" iyy="0.0005843" izz="0.0031631"
-             ixy="0.000" iyz="0.000" ixz="0.000" />
+             ixy="0.000" iyz="0.000" ixz="0.000" /-->
   </xacro:macro>
   <!-- arm_3 -->
@@ -69,8 +73,10 @@
   <xacro:macro name="arm_3_inertial" >
     <mass value="0.821" />
-    <origin xyz="0.000 0.104 0.020"
+    <inertia ixx="0.001" iyy="0.001" izz="0.001"
+             ixy="0.000" iyz="0.000" ixz="0.000" />
+    <!-- origin xyz="0.000 0.104 0.020"
             rpy="0 0 ${M_PI * (90 / 180)}"/>
     <inertia ixx="0.00172767" iyy="0.00041967" izz="0.0018468"
-             ixy="0.000" iyz="0.000" ixz="0.000" />
+             ixy="0.000" iyz="0.000" ixz="0.000" /-->
   </xacro:macro>
   <!-- arm_4 -->
@@ -85,8 +91,10 @@
   <xacro:macro name="arm_4_inertial" >
     <mass value="0.769" />
-    <origin xyz="0.000 0.054 -0.025"
+    <inertia ixx="0.001" iyy="0.001" izz="0.001"
+             ixy="0.000" iyz="0.000" ixz="0.000" />
+    <!-- origin xyz="0.000 0.054 -0.025"
             rpy="${M_PI * (40 / 180)} ${M_PI * (180 / 180)} 0"/>
     <inertia ixx="0.0006764" iyy="0.0010573" izz="0.0006610"
-             ixy="0.000" iyz="0.000" ixz="0.000" />
+             ixy="0.000" iyz="0.000" ixz="0.000" /-->
   </xacro:macro>
   <!-- arm_5 -->
@@ -101,8 +109,10 @@
   <xacro:macro name="arm_5_inertial" >
     <mass value="0.687" />
-    <origin xyz="0.000 0.001 -0.016"
+    <inertia ixx="0.001" iyy="0.001" izz="0.001"
+             ixy="0.000" iyz="0.000" ixz="0.000" />
+    <!-- origin xyz="0.000 0.001 -0.016"
             rpy="0 ${M_PI * (90 / 180)} 0"/>
     <inertia ixx="0.0001934" iyy="0.0001602" izz="0.0000689"
-             ixy="0.000" iyz="0.000" ixz="0.000" />
+             ixy="0.000" iyz="0.000" ixz="0.000" /-->
   </xacro:macro>
   <!-- gripper_base -->
@@ -115,8 +125,10 @@
   <xacro:property name="gripper_base_link_mass" value="0.199" />
   <xacro:macro name="gripper_base_inertia" >
-    <origin xyz="0.000 0.000 0.029"
+    <inertia ixx="0.001" iyy="0.001" izz="0.001"
+             ixy="0.000" iyz="0.000" ixz="0.000" />
+    <!-- origin xyz="0.000 0.000 0.029"
             rpy="0 ${M_PI * (180 / 180)} ${M_PI * (90 / 180)}"/>
     <inertia ixx="0.0002324" iyy="0.0003629" izz="0.0002067"
-             ixy="0.000" iyz="0.000" ixz="0.000" />
+             ixy="0.000" iyz="0.000" ixz="0.000" /-->
   </xacro:macro>
   <!-- fingers paramaters -->

File: youbot_description/urdf/youbot.urdf.xacro (robot description, xacro)
@@ -4,5 +4,5 @@
   <xacro:property name="M_PI" value="3.1415926535897931"/>
   <!-- used for having a more realistic behavior -->
-  <xacro:property name="effort_correct" value="10.0" />
+  <xacro:property name="effort_correct" value="100.0" />
   <!-- Import the spec provided by youBot store -->
   <xacro:include filename="$(find youbot_description)/urdf/spec.urdf.xacro"/>
