Commit message: revert to real values

File: youbot_description/urdf/spec.urdf.xacro (robot description, xacro)
@@ -76,9 +76,4 @@
              ixy="0.000" iyz="0.000" ixz="0.000" />
     <!-- origin xyz="0.000 0.104 0.020"
-            rpy="0 0 ${M_PI * (90 / 180)}"/>
-    <inertia ixx="0.00172767" iyy="0.00041967" izz="0.0018468"
-             ixy="0.000" iyz="0.000" ixz="0.000" /-->
-  </xacro:macro>
-  <!-- arm_4 -->
   <xacro:macro name="arm_4_joint" >
     <origin xyz="0.000 0.135 0.000"
@@ -91,10 +86,8 @@
   <xacro:macro name="arm_4_inertial" >
     <mass value="0.769" />
-    <inertia ixx="0.001" iyy="0.001" izz="0.001"
-             ixy="0.000" iyz="0.000" ixz="0.000" />
-    <!-- origin xyz="0.000 0.054 -0.025"
+    <origin xyz="0.000 0.054 -0.025"
             rpy="${M_PI * (40 / 180)} ${M_PI * (180 / 180)} 0"/>
     <inertia ixx="0.0006764" iyy="0.0010573" izz="0.0006610"
-             ixy="0.000" iyz="0.000" ixz="0.000" /-->
+             ixy="0.000" iyz="0.000" ixz="0.000" />
   </xacro:macro>
   <!-- arm_5 -->
@@ -109,10 +102,8 @@
   <xacro:macro name="arm_5_inertial" >
     <mass value="0.687" />
-    <inertia ixx="0.001" iyy="0.001" izz="0.001"
-             ixy="0.000" iyz="0.000" ixz="0.000" />
-    <!-- origin xyz="0.000 0.001 -0.016"
+    <origin xyz="0.000 0.001 -0.016"
             rpy="0 ${M_PI * (90 / 180)} 0"/>
     <inertia ixx="0.0001934" iyy="0.0001602" izz="0.0000689"
-             ixy="0.000" iyz="0.000" ixz="0.000" /-->
+             ixy="0.000" iyz="0.000" ixz="0.000" />
   </xacro:macro>
   <!-- gripper_base -->
@@ -125,10 +116,8 @@
   <xacro:property name="gripper_base_link_mass" value="0.199" />
   <xacro:macro name="gripper_base_inertia" >
-    <inertia ixx="0.001" iyy="0.001" izz="0.001"
-             ixy="0.000" iyz="0.000" ixz="0.000" />
-    <!-- origin xyz="0.000 0.000 0.029"
+    <origin xyz="0.000 0.000 0.029"
             rpy="0 ${M_PI * (180 / 180)} ${M_PI * (90 / 180)}"/>
     <inertia ixx="0.0002324" iyy="0.0003629" izz="0.0002067"
-             ixy="0.000" iyz="0.000" ixz="0.000" /-->
+             ixy="0.000" iyz="0.000" ixz="0.000" />
   </xacro:macro>
   <!-- fingers paramaters -->
@@ -154,2 +143,10 @@
   <xacro:property name="finger_right_link_mass" value="0.010" />
 </robot>
+<?xml version="1.0"?>
+<!-- Copyright 2013 Arn-O. See the LICENSE file at the top-level directory of this distribution and at https://github.com/Arn-O/youbot_ros_tools/blob/master/LICENSE. -->
+<robot name="youbot" xmlns:xacro="http://www.ros.org/wiki/xacro">
+  <!-- TODO: the max value should be a parameter of the robot -->
+  <xacro:property name="finger_right_limit_min" value="0" />
+  <xacro:property name="finger_right_limit_max" value="0.013" />
+  <xacro:property name="finger_right_link_mass" value="0.010" />
+</robot>

File: youbot_description/urdf/youbot.urdf.xacro (robot description, xacro)
@@ -322,4 +322,4 @@
   <xacro:arm_base/>
   <xacro:arm/>
-  <!-- xacro:gripper/ -->
+  <xacro:gripper/>
 </robot>

Commit message: move spec notice

File: youbot_description/urdf/spec.urdf.xacro (robot description, xacro)
@@ -1,4 +1,5 @@
 <?xml version="1.0"?>
 <!-- Copyright 2013 Arn-O. See the LICENSE file at the top-level directory of this distribution and at https://github.com/Arn-O/youbot_ros_tools/blob/master/LICENSE. -->
+<!-- This file should contain parameter provided by the youBot store, see http://www.youbot-store.com/youbot-developers/software/simulation/kuka-youbot-kinematics-dynamics-and-3d-model?c=35. Default parameters should be stored in the robot description directly. -->
 <robot name="youbot" xmlns:xacro="http://www.ros.org/wiki/xacro">
   <!-- base -->
@@ -36,10 +37,8 @@
   <xacro:macro name="arm_1_inertial" >
     <mass value="1.390" />
-    <inertia ixx="0.001" iyy="0.001" izz="0.001"
-             ixy="0.000" iyz="0.000" ixz="0.000" />
-    <!-- origin xyz="0.015 0.004 0.031"
+    <origin xyz="0.015 0.004 0.031"
             rpy="${M_PI * (180 / 180)} ${M_PI * (20 / 180)} 0"/>
     <inertia ixx="0.0029525" iyy="0.0060091" izz="0.0058821"
-             ixy="0.000" iyz="0.000" ixz="0.000" /-->
+             ixy="0.000" iyz="0.000" ixz="0.000" />
   </xacro:macro>
   <!-- arm_2 -->
@@ -55,10 +54,8 @@
   <xacro:macro name="arm_2_inertial" >
     <mass value="1.318" />
-    <inertia ixx="0.001" iyy="0.001" izz="0.001"
-             ixy="0.000" iyz="0.000" ixz="0.000" />
-    <!-- origin xyz="0.114 0.015 -0.019"
+    <origin xyz="0.114 0.015 -0.019"
             rpy="0 ${M_PI * (90 / 180)} ${M_PI * (-90 / 180)}"/>
     <inertia ixx="0.0031145" iyy="0.0005843" izz="0.0031631"
-             ixy="0.000" iyz="0.000" ixz="0.000" /-->
+             ixy="0.000" iyz="0.000" ixz="0.000" />
   </xacro:macro>
   <!-- arm_3 -->
@@ -73,6 +70,10 @@
   <xacro:macro name="arm_3_inertial" >
     <mass value="0.821" />
-    <inertia ixx="0.001" iyy="0.001" izz="0.001"
+    <origin xyz="0.000 0.104 0.020"
+            rpy="0 0 ${M_PI * (90 / 180)}"/>
+    <inertia ixx="0.00172767" iyy="0.00041967" izz="0.0018468"
              ixy="0.000" iyz="0.000" ixz="0.000" />
+  </xacro:macro>
+  <!-- arm_4 -->
   <xacro:macro name="arm_4_joint" >
     <origin xyz="0.000 0.135 0.000"
@@ -142,10 +143,2 @@
   <xacro:property name="finger_right_link_mass" value="0.010" />
 </robot>
-<?xml version="1.0"?>
-<!-- Copyright 2013 Arn-O. See the LICENSE file at the top-level directory of this distribution and at https://github.com/Arn-O/youbot_ros_tools/blob/master/LICENSE. -->
-<robot name="youbot" xmlns:xacro="http://www.ros.org/wiki/xacro">
-  <!-- TODO: the max value should be a parameter of the robot -->
-  <xacro:property name="finger_right_limit_min" value="0" />
-  <xacro:property name="finger_right_limit_max" value="0.013" />
-  <xacro:property name="finger_right_link_mass" value="0.010" />
-</robot>

File: youbot_description/urdf/youbot.urdf.xacro (robot description, xacro)
@@ -1,5 +1,4 @@
 <?xml version="1.0"?>
 <!-- Copyright 2013 Arn-O. See the LICENSE file at the top-level directory of this distribution and at https://github.com/Arn-O/youbot_ros_tools/blob/master/LICENSE. -->
-<!-- This file should contain parameter provided by the youBot store, see http://www.youbot-store.com/youbot-developers/software/simulation/kuka-youbot-kinematics-dynamics-and-3d-model?c=35. Default parameters should be stored in the robot description directly. -->
 <robot xmlns:xacro="http://www.ros.org/wiki/xacro" name="youbot">
   <xacro:property name="M_PI" value="3.1415926535897931"/>

Commit message: nightly build

File: youbot_description/urdf/spec.urdf.xacro (robot description, xacro)
@@ -38,5 +38,5 @@
     <mass value="1.390" />
     <origin xyz="0.015 0.004 0.031"
-            rpy="${M_PI * (180 / 180)} ${M_PI * (20 / 180)} 0"/>
+	    rpy="0 0 ${M_PI * (180 / 180)}" />
     <inertia ixx="0.0029525" iyy="0.0060091" izz="0.0058821"
              ixy="0.000" iyz="0.000" ixz="0.000" />
@@ -55,5 +55,5 @@
     <mass value="1.318" />
     <origin xyz="0.114 0.015 -0.019"
-            rpy="0 ${M_PI * (90 / 180)} ${M_PI * (-90 / 180)}"/>
+	    rpy= "${M_PI * (-90 / 180)} ${M_PI * (90 / 180)} 0"/>
     <inertia ixx="0.0031145" iyy="0.0005843" izz="0.0031631"
              ixy="0.000" iyz="0.000" ixz="0.000" />
@@ -70,6 +70,6 @@
   <xacro:macro name="arm_3_inertial" >
     <mass value="0.821" />
-    <origin xyz="0.000 0.104 0.020"
-            rpy="0 0 ${M_PI * (90 / 180)}"/>
+    <!-- <origin xyz="0.000 0.104 0.020"
+	    rpy="0 0 ${M_PI * (90 / 180)}"/> -->
     <inertia ixx="0.00172767" iyy="0.00041967" izz="0.0018468"
              ixy="0.000" iyz="0.000" ixz="0.000" />

File: youbot_description/urdf/youbot.urdf.xacro (robot description, xacro)
@@ -9,5 +9,4 @@
   <!-- Import all Gazebo-customization elements, including Gazebo colors -->
   <xacro:include filename="$(find youbot_description)/urdf/youbot.gazebo"/>
-  <!-- TODO: change inertia of the base links and the wheels -->
   <xacro:macro name="base">
     <!-- #### base #### -->
@@ -17,5 +16,5 @@
         <mass value="0.001"/>
 	<inertia ixx="0.000001" iyy="0.000001" izz="0.000001"
-	         ixy="0.000" ixz="0.000" iyz="0.000" />
+                 ixy="0.000000" ixz="0.000001" iyz="0.000001" />
       </inertial>
       <visual>
@@ -50,6 +49,6 @@
       <inertial>
         <mass value="${plate_mass}"/>
-	<inertia ixx="0.002" iyy="0.002" izz="0.002"
-	         ixy="0" ixz="0" iyz="0"/>
+	<inertia ixx="0.002000" iyy="0.002000" izz="0.002000"
+	         ixy="0.000000" ixz="0.000000" iyz="0.000000"/>
       </inertial>
       <visual>
@@ -190,5 +189,5 @@
     <!-- ### arm_4 ### -->
     <!-- arm_4 link -->
-    <link name="arm_4_link">
+    <!-- <link name="arm_4_link">
       <inertial>
         <xacro:arm_4_inertial/>
@@ -199,7 +198,7 @@
         </geometry>
       </visual>
-    </link>
+    </link> -->
     <!-- arm_4 joint -->
-    <joint name="arm_4_joint" type="revolute">
+    <!-- <joint name="arm_4_joint" type="revolute">
       <xacro:arm_4_joint/>
       <child link="arm_4_link"/>
@@ -212,8 +211,8 @@
         <mechanicalReduction>1</mechanicalReduction>
       </actuator>
-    </transmission>
+    </transmission> -->
     <!-- ### arm_5 ### -->
     <!-- arm_5 link -->
-    <link name="arm_5_link">
+    <!-- <link name="arm_5_link">
       <inertial>
         <xacro:arm_5_inertial/>
@@ -224,7 +223,7 @@
         </geometry>
       </visual>
-    </link>
+    </link> -->
     <!-- arm_5 joint -->
-    <joint name="arm_5_joint" type="revolute">
+    <!-- <joint name="arm_5_joint" type="revolute">
       <xacro:arm_5_joint/>
       <child link="arm_5_link"/>
@@ -237,5 +236,5 @@
         <mechanicalReduction>1</mechanicalReduction>
       </actuator>
-    </transmission>
+    </transmission> -->
   </xacro:macro>
   <xacro:macro name="gripper">

Commit message: simplified inertia

File: youbot_description/urdf/spec.urdf.xacro (robot description, xacro)
@@ -37,8 +37,11 @@
   <xacro:macro name="arm_1_inertial" >
     <mass value="1.390" />
-    <origin xyz="0.015 0.004 0.031"
+    <origin xyz="0.000 0.000 0.057"/>
+    <inertia ixx="0.000578" iyy="0.000579" izz="0.001821"
+	     ixy="0.000" iyz="0.000" ixz="0.000" /> -->
+    <!-- <origin xyz="0.015 0.004 0.031"
 	    rpy="0 0 ${M_PI * (180 / 180)}" />
     <inertia ixx="0.0029525" iyy="0.0060091" izz="0.0058821"
-             ixy="0.000" iyz="0.000" ixz="0.000" />
+	     ixy="0.000" iyz="0.000" ixz="0.000" /> -->
   </xacro:macro>
   <!-- arm_2 -->
@@ -54,8 +57,11 @@
   <xacro:macro name="arm_2_inertial" >
     <mass value="1.318" />
-    <origin xyz="0.114 0.015 -0.019"
+    <origin xyz="0.016 0.000 0.000"/>
+    <inertia ixx="0.000394" iyy="0.000549" izz="0.000549"
+	     ixy="0.000" iyz="0.000" ixz="0.000" />
+    <!-- <origin xyz="0.114 0.015 -0.019"
 	    rpy= "${M_PI * (-90 / 180)} ${M_PI * (90 / 180)} 0"/>
     <inertia ixx="0.0031145" iyy="0.0005843" izz="0.0031631"
-             ixy="0.000" iyz="0.000" ixz="0.000" />
+	     ixy="0.000" iyz="0.000" ixz="0.000" /> -->
   </xacro:macro>
   <!-- arm_3 -->

File: youbot_description/urdf/youbot.urdf.xacro (robot description, xacro)
@@ -164,5 +164,5 @@
     <!-- ### arm_3 ### -->
     <!-- arm_3 link -->
-    <link name="arm_3_link">
+    <!-- <link name="arm_3_link">
       <inertial>
         <xacro:arm_3_inertial/>
@@ -173,7 +173,7 @@
         </geometry>
       </visual>
-    </link>
+    </link> -->
     <!-- arm_3 joint -->
-    <joint name="arm_3_joint" type="revolute">
+    <!-- <joint name="arm_3_joint" type="revolute">
       <xacro:arm_3_joint/>
       <child link="arm_3_link"/>
@@ -186,5 +186,5 @@
         <mechanicalReduction>1</mechanicalReduction>
       </actuator>
-    </transmission>
+    </transmission> -->
     <!-- ### arm_4 ### -->
     <!-- arm_4 link -->

Commit message: simplified inertia

File: youbot_description/urdf/spec.urdf.xacro (robot description, xacro)
@@ -57,6 +57,6 @@
   <xacro:macro name="arm_2_inertial" >
     <mass value="1.318" />
-    <origin xyz="0.016 0.000 0.000"/>
-    <inertia ixx="0.000394" iyy="0.000549" izz="0.000549"
+    <origin xyz="0.077 0.000 0.000"/>
+    <inertia ixx="0.002913" iyy="0.000549" izz="0.000549"
 	     ixy="0.000" iyz="0.000" ixz="0.000" />
     <!-- <origin xyz="0.114 0.015 -0.019"
@@ -76,8 +76,11 @@
   <xacro:macro name="arm_3_inertial" >
     <mass value="0.821" />
-    <!-- <origin xyz="0.000 0.104 0.020"
-	    rpy="0 0 ${M_PI * (90 / 180)}"/> -->
+    <origin xyz="0.000 0.067 0.000"/>
+    <inertia ixx="0.000342" iyy="0.001418" izz="0.000342"
+             ixy="0.000" iyz="0.000" ixz="0.000" />
+     <!-- <origin xyz="0.000 0.104 0.020"
+	    rpy="0 0 ${M_PI * (90 / 180)}"/>
     <inertia ixx="0.00172767" iyy="0.00041967" izz="0.0018468"
-             ixy="0.000" iyz="0.000" ixz="0.000" />
+	     ixy="0.000" iyz="0.000" ixz="0.000" /> -->
   </xacro:macro>
   <!-- arm_4 -->

File: youbot_description/urdf/youbot.urdf.xacro (robot description, xacro)
@@ -164,5 +164,5 @@
     <!-- ### arm_3 ### -->
     <!-- arm_3 link -->
-    <!-- <link name="arm_3_link">
+    <link name="arm_3_link">
       <inertial>
         <xacro:arm_3_inertial/>
@@ -173,7 +173,7 @@
         </geometry>
       </visual>
-    </link> -->
+    </link>
     <!-- arm_3 joint -->
-    <!-- <joint name="arm_3_joint" type="revolute">
+    <joint name="arm_3_joint" type="revolute">
       <xacro:arm_3_joint/>
       <child link="arm_3_link"/>
@@ -186,5 +186,5 @@
         <mechanicalReduction>1</mechanicalReduction>
       </actuator>
-    </transmission> -->
+    </transmission>
     <!-- ### arm_4 ### -->
     <!-- arm_4 link -->

Commit message: simplified inertia

File: youbot_description/urdf/spec.urdf.xacro (robot description, xacro)
@@ -95,8 +95,11 @@
   <xacro:macro name="arm_4_inertial" >
     <mass value="0.769" />
-    <origin xyz="0.000 0.054 -0.025"
+    <origin xyz="0.000 0.057 0.000"/>
+    <inertia ixx="0.000320" iyy="0.000993" izz="0.000320"
+             ixy="0.000" iyz="0.000" ixz="0.000" />
+     <!-- <origin xyz="0.000 0.054 -0.025"
             rpy="${M_PI * (40 / 180)} ${M_PI * (180 / 180)} 0"/>
     <inertia ixx="0.0006764" iyy="0.0010573" izz="0.0006610"
-             ixy="0.000" iyz="0.000" ixz="0.000" />
+	     ixy="0.000" iyz="0.000" ixz="0.000" /> -->
   </xacro:macro>
   <!-- arm_5 -->
@@ -111,8 +114,11 @@
   <xacro:macro name="arm_5_inertial" >
     <mass value="0.687" />
-    <origin xyz="0.000 0.001 -0.016"
+    <origin xyz="0.000 0.000 0.000"/>
+    <inertia ixx="0.000247" iyy="0.000247" izz="0.000247"
+             ixy="0.000" iyz="0.000" ixz="0.000" />
+     <!-- <origin xyz="0.000 0.001 -0.016"
             rpy="0 ${M_PI * (90 / 180)} 0"/>
     <inertia ixx="0.0001934" iyy="0.0001602" izz="0.0000689"
-             ixy="0.000" iyz="0.000" ixz="0.000" />
+	     ixy="0.000" iyz="0.000" ixz="0.000" /> -->
   </xacro:macro>
   <!-- gripper_base -->
@@ -125,8 +131,11 @@
   <xacro:property name="gripper_base_link_mass" value="0.199" />
   <xacro:macro name="gripper_base_inertia" >
-    <origin xyz="0.000 0.000 0.029"
+    <origin xyz="0.000 0.000 0.000"/>
+    <inertia ixx="0.000072" iyy="0.000072" izz="0.000072"
+             ixy="0.000" iyz="0.000" ixz="0.000" />
+     <!-- <origin xyz="0.000 0.000 0.029"
             rpy="0 ${M_PI * (180 / 180)} ${M_PI * (90 / 180)}"/>
     <inertia ixx="0.0002324" iyy="0.0003629" izz="0.0002067"
-             ixy="0.000" iyz="0.000" ixz="0.000" />
+	     ixy="0.000" iyz="0.000" ixz="0.000" /> -->
   </xacro:macro>
   <!-- fingers paramaters -->

File: youbot_description/urdf/youbot.urdf.xacro (robot description, xacro)
@@ -189,5 +189,5 @@
     <!-- ### arm_4 ### -->
     <!-- arm_4 link -->
-    <!-- <link name="arm_4_link">
+    <link name="arm_4_link">
       <inertial>
         <xacro:arm_4_inertial/>
@@ -198,7 +198,7 @@
         </geometry>
       </visual>
-    </link> -->
+    </link>
     <!-- arm_4 joint -->
-    <!-- <joint name="arm_4_joint" type="revolute">
+    <joint name="arm_4_joint" type="revolute">
       <xacro:arm_4_joint/>
       <child link="arm_4_link"/>
@@ -211,8 +211,8 @@
         <mechanicalReduction>1</mechanicalReduction>
       </actuator>
-    </transmission> -->
+    </transmission>
     <!-- ### arm_5 ### -->
     <!-- arm_5 link -->
-    <!-- <link name="arm_5_link">
+    <link name="arm_5_link">
       <inertial>
         <xacro:arm_5_inertial/>
@@ -223,7 +223,7 @@
         </geometry>
       </visual>
-    </link> -->
+    </link>
     <!-- arm_5 joint -->
-    <!-- <joint name="arm_5_joint" type="revolute">
+    <joint name="arm_5_joint" type="revolute">
       <xacro:arm_5_joint/>
       <child link="arm_5_link"/>
@@ -236,5 +236,5 @@
         <mechanicalReduction>1</mechanicalReduction>
       </actuator>
-    </transmission> -->
+    </transmission>
   </xacro:macro>
   <xacro:macro name="gripper">
@@ -264,5 +264,6 @@
       <inertial>
         <mass value="${finger_left_link_mass}"/>
-        <inertia ixx="0.00001" ixy="0.000" ixz="0.000" iyy="0.00001" iyz="0.00001" izz="0.00001"/>
+	<inertia ixx="0.000100" iyy="0.000100" izz="0.000100"
+		 ixy="0.000000" ixz="0.000000" iyz="0.000000"/>
       </inertial>
       <visual>
@@ -294,5 +295,6 @@
       <inertial>
         <mass value="${finger_right_link_mass}"/>
-        <inertia ixx="0.00001" ixy="0.000" ixz="0.000" iyy="0.00001" iyz="0.00001" izz="0.00001"/>
+	<inertia ixx="0.000100" iyy="0.000100" izz="0.000100"
+	         ixy="0.000000" ixz="0.000000" iyz="0.000000"/>
       </inertial>
       <visual>
@@ -326,4 +328,4 @@
   <xacro:arm_base/>
   <xacro:arm/>
-  <!-- xacro:gripper/ -->
+  <xacro:gripper/>
 </robot>
