Commit message: massive merge

File: youbot_description/urdf/youbot.urdf.xacro (robot description, xacro)
@@ -2,8 +2,11 @@
 <!-- Refactored by Arn-O -->
 <robot name="youbot" xmlns:xacro="http://www.ros.org/wiki/xacro">
-  <!-- includes -->
+  <property name="M_PI" value="3.1415926535897931" />
+  <!-- Casters -->
+  <property name="cal_caster_fl" value="0.0" />
+  <property name="cal_caster_fr" value="0.0" />
+  <property name="cal_caster_bl" value="0.0" />
+  <property name="cal_caster_br" value="0.0" />
   <xacro:include filename="$(find youbot_description)/urdf/specs.urdf.xacro" />
-  <!-- xacro:include filename="$(find youbot_description)/urdf/youbot_base/base.gazebo.xacro" /-->
-  <xacro:macro name="youbot_base">
     <!-- ### links ### -->
     <!-- base -->
@@ -99,5 +102,52 @@
       </collision>
     </link>
+  <!-- plate -->
+  <link name="plate_link">
+    <inertial>
+     <mass value="${plate_mass}"/>
+     <inertia ixx="0.01" ixy="0" ixz="0" iyy="0.01" iyz="0" izz="0.01" />
+    </inertial>
+    <visual>
+      <geometry>
+        <mesh filename="package://youbot_description/meshes/youbot_plate/plate.dae" />
+      </geometry>
+    </visual>
+  </link>
+  <!-- arm -->
+    <link name="arm_base_link">
+      <inertial>
+        <mass value="${arm_base_mass}" />
+        <inertia ixx="0.010" ixy="0.000" ixz="0.000" iyy="0.010" iyz="0.000" izz="0.010" />
+      </inertial>
+      <visual>
+        <geometry>
+          <mesh filename="package://youbot_description/meshes/youbot_arm/arm_base_frame.dae"/>
+        </geometry>
+      </visual>
+    </link>
+    <link name="arm_1_link">
+      <inertial>
+        <mass value="${arm_1_link_mass}" />
+        <inertia ixx="0.010" ixy="0.000" ixz="0.000" iyy="0.010" iyz="0.000" izz="0.010" />
+      </inertial>
+      <visual>
+        <geometry>
+          <mesh filename="package://youbot_description/meshes/youbot_arm/arm_joint_1.dae"/>
+        </geometry>
+      </visual>
+    </link>
+    <link name="arm_2_link">
+      <inertial>
+        <mass value="${arm_2_link_mass}" />
+        <inertia ixx="0.010" ixy="0.000" ixz="0.000" iyy="0.010" iyz="0.000" izz="0.010" />
+      </inertial>
+      <visual>
+        <geometry>
+          <mesh filename="package://youbot_description/meshes/youbot_arm/arm_joint_2.dae"/>
+        </geometry>
+      </visual>
+    </link>
     <!-- ### joints ### -->
+  <!-- base -->
     <joint name="base_joint" type="fixed">
       <origin xyz="${base_pose_x} ${base_pose_y} ${base_pose_z}" rpy="0 0 0" />
@@ -125,6 +175,34 @@
       <child link="wheel_link_br" />
     </joint>
+    <joint name="arm_base_joint" type="fixed">
+      <origin xyz="${arm_base_pose_x} ${arm_base_pose_y} ${arm_base_pose_z}" rpy="0 0 0" />
+      <parent link="base_link"/>
+      <child link="arm_base_link" />
+    </joint>
+  <!-- arm -->
+    <joint name="arm_1_joint" type="revolute">
+      <origin xyz="${arm_1_link_pose_x} ${arm_1_link_pose_y} ${arm_1_link_pose_z}"
+              rpy="${arm_1_link_orient_r} ${arm_1_link_orient_p} ${arm_1_link_orient_y}" />
+      <parent link="arm_base_link"/>
+      <child link="arm_1_link" />
+      <limit lower="-2.0" upper="2.0" effort="1000" velocity="3" />
+    </joint>
+    <joint name="arm_2_joint" type="revolute">
+      <origin xyz="${arm_2_link_pose_x} ${arm_2_link_pose_y} ${arm_2_link_pose_z}"
+              rpy="${arm_2_link_orient_r} ${arm_2_link_orient_p} ${arm_2_link_orient_y}" />
+      <parent link="arm_1_link"/>
+      <child link="arm_2_link" />
+      <limit lower="-2.0" upper="2.0" effort="1000" velocity="3" />
+    </joint>
     <!-- extensions -->
-    <xacro:youbot_base_gazebo />
-  </xacro:macro>
+    <!-- uncomment for adding the controllers -->
+    <!-- xacro:youbot_arm_transmission /-->
+  <!-- youbot base -->
+  <xacro:include filename="$(find youbot_description)/urdf/youbot_base/base.urdf.xacro" />
+  <!-- youbot plate -->
+  <xacro:include filename="$(find youbot_description)/urdf/youbot_plate/plate.urdf.xacro" />
+  <!-- generic simulator_gazebo plugins for starting mechanism control, ros time, ros battery -->
+  <xacro:include filename="$(find youbot_description)/gazebo/gazebo.urdf.xacro" />
+  <xacro:youbot_base />
+  <xacro:youbot_plate />
 </robot>

Commit message: nightly build

File: youbot_description/urdf/youbot.urdf.xacro (robot description, xacro)
@@ -2,11 +2,7 @@
 <!-- Refactored by Arn-O -->
 <robot name="youbot" xmlns:xacro="http://www.ros.org/wiki/xacro">
-  <property name="M_PI" value="3.1415926535897931" />
-  <!-- Casters -->
-  <property name="cal_caster_fl" value="0.0" />
-  <property name="cal_caster_fr" value="0.0" />
-  <property name="cal_caster_bl" value="0.0" />
-  <property name="cal_caster_br" value="0.0" />
-  <xacro:include filename="$(find youbot_description)/urdf/specs.urdf.xacro" />
+  <xacro:property name="M_PI" value="3.1415926535897931" />
+  <xacro:include filename="$(find youbot_description)/urdf/spec.urdf.xacro" />
+  <xacro:macro name="youbot_description" >
     <!-- ### links ### -->
     <!-- base -->
@@ -29,9 +25,10 @@
       <visual>
         <geometry>
-          <mesh filename="package://youbot_description/meshes/youbot_base/base_frame.dae"/>
+          <mesh filename="package://youbot_description/meshes/base_frame.dae"/>
         </geometry>
       </visual>
     </link>
     <!-- wheels -->
+    <!-- TODO: replace the following 4 code blocks by macros -->
     <!-- front left wheel -->
     <link name="wheel_link_fl">
@@ -102,5 +99,5 @@
       </collision>
     </link>
-  <!-- plate -->
+  <!-- plate links -->
   <link name="plate_link">
     <inertial>
@@ -110,9 +107,9 @@
     <visual>
       <geometry>
-        <mesh filename="package://youbot_description/meshes/youbot_plate/plate.dae" />
+        <mesh filename="package://youbot_description/meshes/plate.dae" />
       </geometry>
     </visual>
   </link>
-  <!-- arm -->
+  <!-- arm_base link -->
     <link name="arm_base_link">
       <inertial>
@@ -122,8 +119,9 @@
       <visual>
         <geometry>
-          <mesh filename="package://youbot_description/meshes/youbot_arm/arm_base_frame.dae"/>
-        </geometry>
-      </visual>
-    </link>
+          <mesh filename="package://youbot_description/meshes/arm_base_frame.dae"/>
+        </geometry>
+      </visual>
+    </link>
+  <!-- arm_1 link -->
     <link name="arm_1_link">
       <inertial>
@@ -132,9 +130,11 @@
       </inertial>
       <visual>
-        <geometry>
-          <mesh filename="package://youbot_description/meshes/youbot_arm/arm_joint_1.dae"/>
-        </geometry>
-      </visual>
-    </link>
+        <origin xyz="0 0 0" rpy="${arm_1_link_orient_r} ${arm_1_link_orient_p} ${arm_1_link_orient_y}" />
+        <geometry>
+          <mesh filename="package://youbot_description/meshes/arm_joint_1.dae"/>
+        </geometry>
+      </visual>
+    </link>
+  <!-- arm_2 link -->
     <link name="arm_2_link">
       <inertial>
@@ -143,11 +143,12 @@
       </inertial>
       <visual>
-        <geometry>
-          <mesh filename="package://youbot_description/meshes/youbot_arm/arm_joint_2.dae"/>
+        <origin xyz="0 0 0" rpy="${arm_2_link_orient_r} ${arm_2_link_orient_p} ${arm_2_link_orient_y}" />
+        <geometry>
+          <mesh filename="package://youbot_description/meshes/arm_joint_2.dae"/>
         </geometry>
       </visual>
     </link>
     <!-- ### joints ### -->
-  <!-- base -->
+  <!-- base joint -->
     <joint name="base_joint" type="fixed">
       <origin xyz="${base_pose_x} ${base_pose_y} ${base_pose_z}" rpy="0 0 0" />
@@ -155,4 +156,5 @@
       <child link="base_link" />
     </joint>
+  <!-- wheels joints -->
     <joint name="wheel_fl_joint" type="fixed">
       <origin xyz="${wheel_fl_pose_x} ${wheel_fl_pose_y} ${wheel_fl_pose_z}" rpy="0 0 0" />
@@ -175,4 +177,11 @@
       <child link="wheel_link_br" />
     </joint>
+<!-- plate joint -->
+    <joint name="plate_joint" type="fixed">
+      <origin xyz="${arm_base_pose_x} ${arm_base_pose_y} ${arm_base_pose_z}" rpy="0 0 0" />
+      <parent link="base_link"/>
+      <child link="plate_link" />
+    </joint>
+  <!-- arm_base joint -->
     <joint name="arm_base_joint" type="fixed">
       <origin xyz="${arm_base_pose_x} ${arm_base_pose_y} ${arm_base_pose_z}" rpy="0 0 0" />
@@ -180,29 +189,24 @@
       <child link="arm_base_link" />
     </joint>
-  <!-- arm -->
+  <!-- arm_1 joint -->
     <joint name="arm_1_joint" type="revolute">
-      <origin xyz="${arm_1_link_pose_x} ${arm_1_link_pose_y} ${arm_1_link_pose_z}"
-              rpy="${arm_1_link_orient_r} ${arm_1_link_orient_p} ${arm_1_link_orient_y}" />
+      <origin xyz="${arm_1_link_pose_x} ${arm_1_link_pose_y} ${arm_1_link_pose_z}" />
       <parent link="arm_base_link"/>
       <child link="arm_1_link" />
+      <axis xyz="0 0 1" />
       <limit lower="-2.0" upper="2.0" effort="1000" velocity="3" />
     </joint>
+  <!-- arm_2 joint -->
     <joint name="arm_2_joint" type="revolute">
-      <origin xyz="${arm_2_link_pose_x} ${arm_2_link_pose_y} ${arm_2_link_pose_z}"
-              rpy="${arm_2_link_orient_r} ${arm_2_link_orient_p} ${arm_2_link_orient_y}" />
+      <origin xyz="${arm_2_link_pose_x} ${arm_2_link_pose_y} ${arm_2_link_pose_z}" />
       <parent link="arm_1_link"/>
       <child link="arm_2_link" />
+      <axis xyz="0 1 0" />
       <limit lower="-2.0" upper="2.0" effort="1000" velocity="3" />
     </joint>
+  </xacro:macro>
+  <xacro:youbot_description />
     <!-- extensions -->
     <!-- uncomment for adding the controllers -->
     <!-- xacro:youbot_arm_transmission /-->
-  <!-- youbot base -->
-  <xacro:include filename="$(find youbot_description)/urdf/youbot_base/base.urdf.xacro" />
-  <!-- youbot plate -->
-  <xacro:include filename="$(find youbot_description)/urdf/youbot_plate/plate.urdf.xacro" />
-  <!-- generic simulator_gazebo plugins for starting mechanism control, ros time, ros battery -->
-  <xacro:include filename="$(find youbot_description)/gazebo/gazebo.urdf.xacro" />
-  <xacro:youbot_base />
-  <xacro:youbot_plate />
 </robot>

Commit message: fix eol

File: youbot_description/urdf/youbot.urdf.xacro (robot description, xacro)
@@ -250,5 +250,5 @@
     <joint name="gripper_base_joint" type="fixed">
       <origin xyz="${gripper_base_link_pose_x} ${gripper_base_link_pose_y} ${gripper_base_link_pose_z}"
-              rpy="${gripper_base_link_orient_r} ${gripper_base_link_orient_p}                                             ${gripper_base_link_orient_y}"/>
+              rpy="${gripper_base_link_orient_r} ${gripper_base_link_orient_p} ${gripper_base_link_orient_y}"/>
       <parent link="arm_5_link"/>
       <child link="gripper_base_link"/>
@@ -298,5 +298,5 @@
     <!-- finger_right joint -->
     <joint name="finger_right_joint" type="prismatic">
-      <origin xyz="${finger_right_link_pose_x} ${finger_right_link_pose_y}                                                        ${finger_right_link_pose_z}"/>
+      <origin xyz="${finger_right_link_pose_x} ${finger_right_link_pose_y} ${finger_right_link_pose_z}"/>
       <parent link="gripper_base_link"/>
       <child link="finger_right_link"/>

Commit message: no gripper and pid try

File: youbot_description/urdf/youbot.urdf.xacro (robot description, xacro)
@@ -4,5 +4,5 @@
   <xacro:property name="M_PI" value="3.1415926535897931"/>
   <!-- used for having a more realistic behavior -->
-  <xacro:property name="effort_correct" value="100.0" />
+  <xacro:property name="effort_correct" value="5.0" />
   <!-- Import the spec provided by youBot store -->
   <xacro:include filename="$(find youbot_description)/urdf/spec.urdf.xacro"/>
@@ -321,4 +321,4 @@
   <xacro:arm_base/>
   <xacro:arm/>
-  <xacro:gripper/>
+  <!-- xacro:gripper/ -->
 </robot>

Commit message: inertia for the base

File: youbot_description/urdf/youbot.urdf.xacro (robot description, xacro)
@@ -16,5 +16,6 @@
       <inertial>
         <mass value="0.001"/>
-        <inertia ixx="0.000001" ixy="0.000" ixz="0.000" iyy="0.000001" iyz="0.000" izz="0.000001"/>
+	<inertia ixx="0.000001" iyy="0.000001" izz="0.000001"
+	         ixy="0.000" ixz="0.000" iyz="0.000" />
       </inertial>
       <visual>
@@ -27,6 +28,8 @@
     <link name="base_link">
       <inertial>
-        <mass value="${base_mass}"/>
-        <inertia ixx="0.01" ixy="0.000" ixz="0.000" iyy="0.01" iyz="0.000" izz="0.01"/>
+	<mass value="${base_mass}"/>
+	<!-- cuboid used as an approximation -->
+	<inertia ixx="0.273333" iyy="0.593333" izz="0.801333"
+	         ixy="0.000" ixz="0.000" iyz="0.000"/>
       </inertial>
       <visual>
@@ -47,5 +50,6 @@
       <inertial>
         <mass value="${plate_mass}"/>
-        <inertia ixx="0.002" ixy="0" ixz="0" iyy="0.002" iyz="0" izz="0.002"/>
+	<inertia ixx="0.002" iyy="0.002" izz="0.002"
+	         ixy="0" ixz="0" iyz="0"/>
       </inertial>
       <visual>
@@ -67,5 +71,6 @@
       <inertial>
         <mass value="${wheel_mass}"/>
-        <inertia ixx="0.0014" ixy="0.000" ixz="0.000" iyy="0.0014" iyz="0.000" izz="0.0014"/>
+	<inertia ixx="0.001400" iyy="0.001400" izz="0.001400"
+	         ixy="0.000000" ixz="0.000000" iyz="0.000000"/>
       </inertial>
       <visual>
@@ -100,5 +105,6 @@
     </link>
     <joint name="arm_base_joint" type="fixed">
-      <origin xyz="${arm_base_pose_x} ${arm_base_pose_y} ${arm_base_pose_z}" rpy="0 0 0"/>
+      <origin xyz="${arm_base_pose_x} ${arm_base_pose_y} ${arm_base_pose_z}"
+              rpy="0 0 0"/>
       <parent link="base_link"/>
       <child link="arm_base_link"/>
@@ -321,4 +327,4 @@
   <xacro:arm_base/>
   <xacro:arm/>
-  <xacro:gripper/>
+  <!-- xacro:gripper/ -->
 </robot>

Commit message: plate inertia

File: youbot_description/urdf/youbot.urdf.xacro (robot description, xacro)
@@ -15,6 +15,6 @@
       <inertial>
         <mass value="0.001"/>
-	<inertia ixx="0.000001" iyy="0.000001" izz="0.000001"
-                 ixy="0.000000" ixz="0.000001" iyz="0.000001" />
+	<inertia ixx="0.000100" iyy="0.000100" izz="0.000100"
+                 ixy="0.000000" ixz="0.000001" iyz="0.000000" />
       </inertial>
       <visual>
@@ -49,5 +49,5 @@
       <inertial>
         <mass value="${plate_mass}"/>
-	<inertia ixx="0.002000" iyy="0.002000" izz="0.002000"
+	<inertia ixx="0.057688" iyy="0.029343" izz="0.057688"
 	         ixy="0.000000" ixz="0.000000" iyz="0.000000"/>
       </inertial>

Commit message: backup

File: youbot_description/urdf/youbot.urdf.xacro (robot description, xacro)
@@ -15,5 +15,5 @@
       <inertial>
         <mass value="0.001"/>
-	<inertia ixx="0.000100" iyy="0.000100" izz="0.000100"
+	<inertia ixx="0.000001" iyy="0.000001" izz="0.000001"
                  ixy="0.000000" ixz="0.000001" iyz="0.000000" />
       </inertial>
@@ -30,5 +30,5 @@
 	<!-- cuboid used as an approximation -->
 	<inertia ixx="0.273333" iyy="0.593333" izz="0.801333"
-	         ixy="0.000" ixz="0.000" iyz="0.000"/>
+	 ixy="0.000000" ixz="0.000000" iyz="0.000000"/>
       </inertial>
       <visual>
@@ -50,5 +50,5 @@
         <mass value="${plate_mass}"/>
 	<inertia ixx="0.057688" iyy="0.029343" izz="0.057688"
-	         ixy="0.000000" ixz="0.000000" iyz="0.000000"/>
+		 ixy="0.000000" ixz="0.000000" iyz="0.000000"/>
       </inertial>
       <visual>
@@ -95,5 +95,6 @@
       <inertial>
         <mass value="${arm_base_mass}"/>
-        <inertia ixx="0.010" ixy="0.000" ixz="0.000" iyy="0.010" iyz="0.000" izz="0.010"/>
+	<inertia ixx="0.010000" iyy="0.010000" izz="0.010000"
+	         ixy="0.000000" ixz="0.000000" iyz="0.000000"/>
       </inertial>
       <visual>
@@ -139,5 +140,5 @@
     <!-- ### arm_2 ### -->
     <!-- arm_2 link -->
-    <link name="arm_2_link">
+    <!-- <link name="arm_2_link">
       <inertial>
         <xacro:arm_2_inertial/>
@@ -148,7 +149,7 @@
         </geometry>
       </visual>
-    </link>
+    </link> -->
     <!-- arm_2 joint -->
-    <joint name="arm_2_joint" type="revolute">
+    <!-- <joint name="arm_2_joint" type="revolute">
       <xacro:arm_2_joint/>
       <child link="arm_2_link"/>
@@ -161,8 +162,8 @@
         <mechanicalReduction>1</mechanicalReduction>
       </actuator>
-    </transmission>
+    </transmission> -->
     <!-- ### arm_3 ### -->
     <!-- arm_3 link -->
-    <link name="arm_3_link">
+    <!-- <link name="arm_3_link">
       <inertial>
         <xacro:arm_3_inertial/>
@@ -173,7 +174,7 @@
         </geometry>
       </visual>
-    </link>
+    </link> -->
     <!-- arm_3 joint -->
-    <joint name="arm_3_joint" type="revolute">
+    <!-- <joint name="arm_3_joint" type="revolute">
       <xacro:arm_3_joint/>
       <child link="arm_3_link"/>
@@ -186,8 +187,8 @@
         <mechanicalReduction>1</mechanicalReduction>
       </actuator>
-    </transmission>
+    </transmission> -->
     <!-- ### arm_4 ### -->
     <!-- arm_4 link -->
-    <link name="arm_4_link">
+    <!-- <link name="arm_4_link">
       <inertial>
         <xacro:arm_4_inertial/>
@@ -198,7 +199,7 @@
         </geometry>
       </visual>
-    </link>
+    </link> -->
     <!-- arm_4 joint -->
-    <joint name="arm_4_joint" type="revolute">
+    <!-- <joint name="arm_4_joint" type="revolute">
       <xacro:arm_4_joint/>
       <child link="arm_4_link"/>
@@ -211,8 +212,8 @@
         <mechanicalReduction>1</mechanicalReduction>
       </actuator>
-    </transmission>
+    </transmission> -->
     <!-- ### arm_5 ### -->
     <!-- arm_5 link -->
-    <link name="arm_5_link">
+    <!-- <link name="arm_5_link">
       <inertial>
         <xacro:arm_5_inertial/>
@@ -223,7 +224,7 @@
         </geometry>
       </visual>
-    </link>
+    </link> -->
     <!-- arm_5 joint -->
-    <joint name="arm_5_joint" type="revolute">
+    <!-- <joint name="arm_5_joint" type="revolute">
       <xacro:arm_5_joint/>
       <child link="arm_5_link"/>
@@ -236,5 +237,5 @@
         <mechanicalReduction>1</mechanicalReduction>
       </actuator>
-    </transmission>
+    </transmission> -->
   </xacro:macro>
   <xacro:macro name="gripper">
@@ -328,4 +329,4 @@
   <xacro:arm_base/>
   <xacro:arm/>
-  <xacro:gripper/>
+  <!-- <xacro:gripper/> -->
 </robot>

Commit message: fix render

File: youbot_description/urdf/youbot.urdf.xacro (robot description, xacro)
@@ -140,5 +140,5 @@
     <!-- ### arm_2 ### -->
     <!-- arm_2 link -->
-    <!-- <link name="arm_2_link">
+    <link name="arm_2_link">
       <inertial>
         <xacro:arm_2_inertial/>
@@ -149,7 +149,7 @@
         </geometry>
       </visual>
-    </link> -->
+    </link>
     <!-- arm_2 joint -->
-    <!-- <joint name="arm_2_joint" type="revolute">
+    <joint name="arm_2_joint" type="revolute">
       <xacro:arm_2_joint/>
       <child link="arm_2_link"/>
@@ -162,8 +162,8 @@
         <mechanicalReduction>1</mechanicalReduction>
       </actuator>
-    </transmission> -->
+    </transmission>
     <!-- ### arm_3 ### -->
     <!-- arm_3 link -->
-    <!-- <link name="arm_3_link">
+    <link name="arm_3_link">
       <inertial>
         <xacro:arm_3_inertial/>
@@ -174,7 +174,7 @@
         </geometry>
       </visual>
-    </link> -->
+    </link>
     <!-- arm_3 joint -->
-    <!-- <joint name="arm_3_joint" type="revolute">
+    <joint name="arm_3_joint" type="revolute">
       <xacro:arm_3_joint/>
       <child link="arm_3_link"/>
@@ -187,8 +187,8 @@
         <mechanicalReduction>1</mechanicalReduction>
       </actuator>
-    </transmission> -->
+    </transmission>
     <!-- ### arm_4 ### -->
     <!-- arm_4 link -->
-    <!-- <link name="arm_4_link">
+    <link name="arm_4_link">
       <inertial>
         <xacro:arm_4_inertial/>
@@ -199,7 +199,7 @@
         </geometry>
       </visual>
-    </link> -->
+    </link>
     <!-- arm_4 joint -->
-    <!-- <joint name="arm_4_joint" type="revolute">
+    <joint name="arm_4_joint" type="revolute">
       <xacro:arm_4_joint/>
       <child link="arm_4_link"/>
@@ -212,8 +212,8 @@
         <mechanicalReduction>1</mechanicalReduction>
       </actuator>
-    </transmission> -->
+    </transmission>
     <!-- ### arm_5 ### -->
     <!-- arm_5 link -->
-    <!-- <link name="arm_5_link">
+    <link name="arm_5_link">
       <inertial>
         <xacro:arm_5_inertial/>
@@ -224,7 +224,7 @@
         </geometry>
       </visual>
-    </link> -->
+    </link>
     <!-- arm_5 joint -->
-    <!-- <joint name="arm_5_joint" type="revolute">
+    <joint name="arm_5_joint" type="revolute">
       <xacro:arm_5_joint/>
       <child link="arm_5_link"/>
@@ -237,5 +237,5 @@
         <mechanicalReduction>1</mechanicalReduction>
       </actuator>
-    </transmission> -->
+    </transmission>
   </xacro:macro>
   <xacro:macro name="gripper">
@@ -329,4 +329,4 @@
   <xacro:arm_base/>
   <xacro:arm/>
-  <!-- <xacro:gripper/> -->
+  <xacro:gripper/>
 </robot>

Commit message: fix color render

File: youbot_description/urdf/youbot.urdf.xacro (robot description, xacro)
@@ -269,6 +269,7 @@
       </inertial>
       <visual>
-        <geometry>
-          <mesh filename="package://youbot_description/meshes/gripper_left_finger.dae"/>
+	<origin rpy="0 0 ${M_PI}" />
+	<geometry>
+          <mesh filename="package://youbot_description/meshes/gripper_right_finger.dae"/>
         </geometry>
       </visual>
