Commit message: investigate issue #1

File: youbot_description/urdf/youbot.urdf.xacro (robot description, xacro)
@@ -140,5 +140,5 @@
     <!-- ### arm_2 ### -->
     <!-- arm_2 link -->
-    <link name="arm_2_link">
+    <!-- link name="arm_2_link">
       <inertial>
         <xacro:arm_2_inertial/>
@@ -149,7 +149,7 @@
         </geometry>
       </visual>
-    </link>
+    </link -->
     <!-- arm_2 joint -->
-    <joint name="arm_2_joint" type="revolute">
+    <!-- joint name="arm_2_joint" type="revolute">
       <xacro:arm_2_joint/>
       <child link="arm_2_link"/>
@@ -162,8 +162,8 @@
         <mechanicalReduction>1</mechanicalReduction>
       </actuator>
-    </transmission>
+    </transmission -->
     <!-- ### arm_3 ### -->
     <!-- arm_3 link -->
-    <link name="arm_3_link">
+    <!-- link name="arm_3_link">
       <inertial>
         <xacro:arm_3_inertial/>
@@ -174,7 +174,7 @@
         </geometry>
       </visual>
-    </link>
+    </link -->
     <!-- arm_3 joint -->
-    <joint name="arm_3_joint" type="revolute">
+    <!-- joint name="arm_3_joint" type="revolute">
       <xacro:arm_3_joint/>
       <child link="arm_3_link"/>
@@ -187,8 +187,8 @@
         <mechanicalReduction>1</mechanicalReduction>
       </actuator>
-    </transmission>
+    </transmission -->
     <!-- ### arm_4 ### -->
     <!-- arm_4 link -->
-    <link name="arm_4_link">
+    <!-- link name="arm_4_link">
       <inertial>
         <xacro:arm_4_inertial/>
@@ -199,7 +199,7 @@
         </geometry>
       </visual>
-    </link>
+    </link -->
     <!-- arm_4 joint -->
-    <joint name="arm_4_joint" type="revolute">
+    <!-- joint name="arm_4_joint" type="revolute">
       <xacro:arm_4_joint/>
       <child link="arm_4_link"/>
@@ -212,8 +212,8 @@
         <mechanicalReduction>1</mechanicalReduction>
       </actuator>
-    </transmission>
+    </transmission -->
     <!-- ### arm_5 ### -->
     <!-- arm_5 link -->
-    <link name="arm_5_link">
+    <!-- link name="arm_5_link">
       <inertial>
         <xacro:arm_5_inertial/>
@@ -224,7 +224,7 @@
         </geometry>
       </visual>
-    </link>
+    </link -->
     <!-- arm_5 joint -->
-    <joint name="arm_5_joint" type="revolute">
+    <!-- joint name="arm_5_joint" type="revolute">
       <xacro:arm_5_joint/>
       <child link="arm_5_link"/>
@@ -237,5 +237,5 @@
         <mechanicalReduction>1</mechanicalReduction>
       </actuator>
-    </transmission>
+    </transmission -->
   </xacro:macro>
   <xacro:macro name="gripper">
@@ -330,4 +330,4 @@
   <xacro:arm_base/>
   <xacro:arm/>
-  <xacro:gripper/>
+  <!-- xacro:gripper/ -->
 </robot>
